File: Experimental/KiCad/dib.kicad_sch (KiCad schematic)
At the start: 7 parts, among them X10 10018783-10101TLF, X11 77313-802-20LF, X12 77313-802-20LF, X13 10018783-10101TLF, X14 5051102091, X15 TBP03R1-350-10BE

Commit message: Gerbers update
Parts:
- X10: value 10018783-10101TLF -> 1001878410201TLF; Mouser 649-18783-10101TLF -> 649-1001878410201TLF; TME 1001878310101T-0 -> 1001878410201T-0
Changed lines of the file:
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@@
 	(title_block
 		(title "${project_name}")
-		(date "2025-10-16")
+		(date "2025-10-19")
 		(rev "${project_version}")
 		(company "${project_creator}")
@@
 			)
 		)
-		(property "Value" "10018783-10101TLF"
+		(property "Value" "1001878410201TLF"
 			(at 63.5 107.95 0)
 			(effects
@@
 			)
 		)
-		(property "Mouser" "649-18783-10101TLF"
+		(property "Mouser" "649-1001878410201TLF"
 			(at 53.34 20.32 0)
 			(effects
@@
 			)
 		)
-		(property "TME" "1001878310101T-0"
+		(property "TME" "1001878410201T-0"
 			(at 53.34 20.32 0)
 			(effects
