File: Experimental/KiCad/usb3_hub.kicad_sch (KiCad schematic)
At the start: 75 parts, among them IC10 TPS62933ODRLR, IC11 FUSB303BTMX, IC12 TPS2068E, IC9 USB5816C-I/KD, X6 USB4056-03-A, Y2 VXM7-9032-25M0000000

Commit message: BOM update
Parts:
- C54, C55: value 18p -> 10p; DigiKey 1276-1089-1-ND -> 1276-1069-1-ND; LCSC C1647 -> C318677; Mouser 187-CL10C180JB8NNNC -> 187-CL10C100CB8NNNC; TME CL10C180JB8NNNC -> VJ0603A100JXACW1BC
Changed lines of the file:
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@@
 	(title_block
 		(title "${project_name}")
-		(date "2025-10-15")
+		(date "2025-10-16")
 		(rev "${project_version}")
 		(company "${project_creator}")
 		(comment 1 "${project_license}")
 		(comment 2 "${project_info}")
+		(comment 3 "${project_url}")
 	)
 	(text "Max 3A"
@@
 			)
 		)
-		(property "Value" "18p"
+		(property "Value" "10p"
 			(at 40.64 145.415 90)
 			(effects
@@
 			)
 		)
-		(property "TME" "CL10C180JB8NNNC"
+		(property "TME" "VJ0603A100JXACW1BC"
 			(at 40.64 144.78 0)
 			(effects
@@
 			)
 		)
-		(property "DigiKey" "1276-1089-1-ND"
+		(property "DigiKey" "1276-1069-1-ND"
 			(at 40.64 144.78 0)
 			(effects
@@
 			)
 		)
-		(property "Mouser" "187-CL10C180JB8NNNC"
+		(property "Mouser" "187-CL10C100CB8NNNC"
 			(at 40.64 144.78 0)
 			(effects
@@
 			)
 		)
-		(property "LCSC" "C1647"
+		(property "LCSC" "C318677"
 			(at 40.64 144.78 0)
 			(effects
@@
 			)
 		)
-		(property "Value" "18p"
+		(property "Value" "10p"
 			(at 40.64 155.575 90)
 			(effects
@@
 			)
 		)
-		(property "TME" "CL10C180JB8NNNC"
+		(property "TME" "VJ0603A100JXACW1BC"
 			(at 40.64 154.94 0)
 			(effects
@@
 			)
 		)
-		(property "DigiKey" "1276-1089-1-ND"
+		(property "DigiKey" "1276-1069-1-ND"
 			(at 40.64 154.94 0)
 			(effects
@@
 			)
 		)
-		(property "Mouser" "187-CL10C180JB8NNNC"
+		(property "Mouser" "187-CL10C100CB8NNNC"
 			(at 40.64 154.94 0)
 			(effects
@@
 			)
 		)
-		(property "LCSC" "C1647"
+		(property "LCSC" "C318677"
 			(at 40.64 154.94 0)
 			(effects
