File: Experimental/KiCad/BB3plus test mainboard.kicad_sch (KiCad schematic)
At the start: 13 parts

Commit message: Update project info
Other:
- company: Envox d.o.o. -> ${project_creator}
- title: BB3+ test mainboard -> ${project_name}
Changed lines of the file:
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@@
 	(paper "A4")
 	(title_block
-		(title "BB3+ test mainboard")
-		(date "2025-10-12")
-		(rev "r1B1")
-		(company "Envox d.o.o.")
-		(comment 1 "Licensed under the TAPR Open Hardware License (www.tapr.org/OHL)")
-		(comment 2 "More info at http://www.envox.eu/")
-		(comment 3 "https://github.com/eez-open/eez-bb5-mcu-module")
+		(title "${project_name}")
+		(date "2025-10-13")
+		(rev "${project_version}")
+		(company "${project_creator}")
+		(comment 1 "${project_license}")
+		(comment 2 "${project_info}")
+		(comment 3 "${project_url}")
 	)
 	(junction
