File: Experimental/KiCad/BB3plus test mainboard.kicad_pcb (KiCad board)
At the start: 4 copper layers, 180.5 x 176 mm, 293 parts, among them IC1 SN74HCS02PWR, IC10 TPS62933ODRLR, IC11 FUSB303BTMX, IC12 TPS2068E, IC13 RT9742SNGV, IC14 TPD4E001DRLR, IC15 TPD4E001DRLR, IC16 TPD12S016PWR, IC17 MIC2026A-1YM-TR, IC18 TPD4E001DRLR, IC2 TPS3851H18EDRBR, IC3 M24C32-DFDW6TP, IC4 STM32G071R8T6, IC5 TPA6205A1DGN, IC6 SN74LVC1G14DBVR, IC7 LM64460CPPQRYFRQ1, IC8 TPS62933ODRLR, IC9 USB5816C-I/KD, Q1 DMP3013SFV-7, Q2 2N7002, Q3 2N7002, Q4 MMBT5401, Q5 MMBT5401, Q6 2N7002, Q7 DMP3013SFV-7, Q8 DMP3013SFV-7, SW1 WBL2UOAGQR05CLR, SW2 PEC16-2215F-S0024, X1 1-2199230-6, X10 1001878410201TLF, X11 77313-802-20LF, X12 77313-802-20LF, X13 1001878410201TLF, X14 5051102091, X15 TBP03R1-350-10BE, X3 571-0400, X4 GSP1.9101.1, X5 PJ-002BH-SMT-TR, X6 USB4056-03-A, X7 0862-1J1T-43-F, X8 SS-53000-002, X9 5051102091, Y1 32.768KHz, Y2 VXM7-9032-25M0000000

Commit message: BOM update
Parts:
- Module1: value 2x DF40HC(3.0)-100DS-0.4V(51 -> 2x 10164227-1004A1RLF
Changed lines of the file:
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@@
 			)
 		)
-		(property "Value" "2x DF40HC(3.0)-100DS-0.4V(51"
+		(property "Value" "2x 10164227-1004A1RLF"
 			(at 16.52 0.19 0)
 			(layer "F.Fab")
@@
 			)
 		)
-		(property "DigiKey" "26-DF40HC(3.0)-100DS-0.4V(51)CT-ND"
+		(property "DigiKey" "609-10164227-1004A1RLFCT-ND"
 			(at 0 0 0)
 			(unlocked yes)
@@
 			)
 		)
-		(property "Mouser" "798-DF40HC30100DS451 "
+		(property "Mouser" "649-101642271004RLF"
 			(at 0 0 0)
 			(unlocked yes)
@@
 			)
 		)
-		(property "LCSC" "C424649"
+		(property "LCSC" "C7435219"
 			(at 0 0 0)
 			(unlocked yes)
