File: Experimental/KiCad/misc.kicad_sch (KiCad schematic)
At the start: 79 parts, among them IC6 SN74LVC1G14DBVR, IC7 LM64460CPPQRYFRQ1, IC8 TPS62933ODRLR, Q4 MMBT5401, Q5 2N7002, Q6 DMP3013SFV-7, Q7 DMP3013SFV-7, SW1 WBL2UOAGQR05CLR, SW2 LP4EE1RBATY, SW3 PEC16-2215F-S0024, X3 571-0400, X4 GSP1.9101.1, X5 PJ-002BH-SMT-TR

Commit message: Gerbers update
Parts:
- X3: Label (none) -> PE
Changed lines of the file:
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@@
 	(title_block
 		(title "${project_name}")
-		(date "2025-10-16")
+		(date "2025-10-19")
 		(rev "${project_version}")
 		(company "${project_creator}")
@@
 			)
 		)
+		(property "Label" "PE"
+			(at 27.94 43.18 0)
+			(effects
+				(font
+					(size 0.889 0.889)
+				)
+				(hide yes)
+			)
+		)

Commit message: Replace 3V3 jumper for H7 CM5 with PMOS sw
Parts:
- renumbered C22 to C23, C23 to C24, C24 to C25, C25 to C26, C26 to C27, C27 to C28, C28 to C29, C29 to C30, C30 to C31, C31 to C32, C32 to C33, C33 to C34, C34 to C35, C35 to C36, C36 to C37, C37 to C38, C38 to C39, C39 to C40, C40 to C41, C41 to C42, C42 to C43, C43 to C44, C44 to C45, C45 to C46, C46 to C47, C47 to C48, C48 to C49, C49 to C50, JP13 to JP12, Q4 to Q5, Q5 to Q6, Q6 to Q7, Q7 to Q8, R27 to R28, R28 to R29, R29 to R30, R30 to R31, R31 to R32, R32 to R33, R33 to R34, R34 to R35, R35 to R36, R36 to R37, R37 to R38, R38 to R39, R39 to R40, R40 to R41, R41 to R42, R42 to R43, R43 to R44, R44 to R45, R45 to R46, R46 to R47

Commit message: Jumpers update
Parts:
- renumbered C39 to C38, C38 to C39, C49 to C47, C50 to C48, C47 to C49, C48 to C50, R40 to R39, R39 to R40
Other:
- moved on the sheet: C29, C30, C31, C32, C33, C35, C36, C37, C38, C40, C41, C42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

Commit message: Power switch modified
Parts:
- removed SW2: LP4EE1RBATY, PCM_EEZ_unsorted:LP4XX1RXAXX, symbol PCM_EEZ_unsorted:LP4xx1RxAxx
- renumbered R30 to R28, R28 to R29, R29 to R30, SW3 to SW2
Connections:
- no-connect marks 5 -> 3
Other:
- moved on the sheet: JP12, R28, SW1A, SW1B
