File: KiCad/TFT DSI module/BB3plus DSI TFT display.kicad_pcb (KiCad board)
At the start: 2 copper layers, 136 x 92 mm, 50 parts, among them IC1 AZ1117CH2-3.3TRG1, IC2 TCA9554APWR, IC3 TPS61169DCKR, SW1 B3FS-4052P, SW2 B3FS-4052P, SW3 B3FS-4052P, SW4 B3FS-4052P, X1 5051102091, X2 505110-4091, X3 F3311A7H121010E200

Commit message: TFT display tactile switches footprint correction
Parts:
- SW1, SW2, SW3, SW4: footprint PCM_EEZ_unsorted:B3FS-4052P -> PCM_EEZ_unsorted:B3FS-4052P (cut out)
Other:
- outline, holes or cut-outs redrawn
- board text added: "${project_name} (12/2025 ${project_version})"
- board text removed: "${project_name} (11/2025 ${project_version})"
