File: KiCad/TFT DSI module/BB3plus DSI TFT display.kicad_sch (KiCad schematic)
At the start: 54 parts, among them IC1 AZ1117CH2-3.3TRG1, IC2 TCA9554APWR, IC3 TPS61169DCKR, SW1 B3FS-4052P, SW2 B3FS-4052P, SW3 B3FS-4052P, SW4 B3FS-4052P, X1 5051102091, X2 505110-4091, X3 F3311A7H121010E200

Commit message: TFT display tactile switches footprint correction
Parts:
- C2, C5: DigiKey (none) -> CL21B225KOFNNNG-ND; Mouser (none) -> 187-CL21B225KOFNNNG
- R2, R3: DigiKey (none) -> YAG5344CT-ND; LCSC (none) -> C227988; Mouser (none) -> 603-AC0603FR-075R1L; TME (none) -> AC0603FR-075R1L
- SW1, SW2, SW3, SW4: footprint PCM_EEZ_unsorted:B3FS-4052P -> PCM_EEZ_unsorted:B3FS-4052P (cut out)
Changed lines of the file:
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@@
 	(title_block
 		(title "${project_name}")
-		(date "2025-11-20")
+		(date "2025-11-27")
 		(rev "${project_version}")
 		(company "${project_creator}")
@@
 			)
 		)
-		(property "Footprint" "PCM_EEZ_unsorted:B3FS-4052P"
+		(property "Footprint" "PCM_EEZ_unsorted:B3FS-4052P (cut out)"
 			(at 269.24 91.44 0)
 			(effects
@@
 			)
 		)
-		(property "Footprint" "PCM_EEZ_unsorted:B3FS-4052P"
+		(property "Footprint" "PCM_EEZ_unsorted:B3FS-4052P (cut out)"
 			(at 269.24 132.08 0)
 			(effects
@@
 			)
 		)
-		(property "DigiKey" ""
+		(property "DigiKey" "YAG5344CT-ND"
 			(at 261.62 50.8 0)
 			(effects
@@
 			)
 		)
-		(property "Mouser" ""
+		(property "Mouser" " 603-AC0603FR-075R1L"
 			(at 261.62 50.8 0)
 			(effects
@@
 			)
 		)
-		(property "TME" ""
+		(property "TME" "AC0603FR-075R1L"
 			(at 261.62 50.8 0)
 			(effects
@@
 			)
 		)
-		(property "LCSC" ""
+		(property "LCSC" "C227988"
 			(at 261.62 50.8 0)
 			(effects
@@
 			)
 		)
-		(property "DigiKey" ""
+		(property "DigiKey" "CL21B225KOFNNNG-ND"
 			(at 172.72 71.12 0)
 			(effects
@@
 			)
 		)
-		(property "Mouser" ""
+		(property "Mouser" "187-CL21B225KOFNNNG"
 			(at 172.72 71.12 0)
 			(effects
@@
 			)
 		)
-		(property "Footprint" "PCM_EEZ_unsorted:B3FS-4052P"
+		(property "Footprint" "PCM_EEZ_unsorted:B3FS-4052P (cut out)"
 			(at 269.24 121.92 0)
 			(effects
@@
 			)
 		)
-		(property "Footprint" "PCM_EEZ_unsorted:B3FS-4052P"
+		(property "Footprint" "PCM_EEZ_unsorted:B3FS-4052P (cut out)"
 			(at 269.24 106.68 0)
 			(effects
@@
 			)
 		)
-		(property "DigiKey" ""
+		(property "DigiKey" "YAG5344CT-ND"
 			(at 254 50.8 0)
 			(effects
@@
 			)
 		)
-		(property "Mouser" ""
+		(property "Mouser" " 603-AC0603FR-075R1L"
 			(at 254 50.8 0)
 			(effects
@@
 			)
 		)
-		(property "TME" ""
+		(property "TME" "AC0603FR-075R1L"
 			(at 254 50.8 0)
 			(effects
@@
 			)
 		)
-		(property "LCSC" ""
+		(property "LCSC" "C227988"
 			(at 254 50.8 0)
 			(effects
@@
 			)
 		)
-		(property "DigiKey" ""
+		(property "DigiKey" "CL21B225KOFNNNG-ND"
 			(at 111.76 86.36 0)
 			(effects
@@
 			)
 		)
-		(property "Mouser" ""
+		(property "Mouser" "187-CL21B225KOFNNNG"
 			(at 111.76 86.36 0)
 			(effects

Commit message: Rear panel silkscreen update
Parts:
- R2, R3: DigiKey YAG5344CT-ND -> 13-RT0805FRE075R1LCT-ND; LCSC C227988 -> C364355; Mouser 603-AC0603FR-075R1L -> 603-RT0805FRE075R1L; TME AC0603FR-075R1L -> CRCW08055R10FKTABC
Changed lines of the file:
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@@
 			)
 		)
-		(property "DigiKey" "YAG5344CT-ND"
+		(property "DigiKey" "13-RT0805FRE075R1LCT-ND"
 			(at 261.62 50.8 0)
 			(effects
@@
 			)
 		)
-		(property "Mouser" " 603-AC0603FR-075R1L"
+		(property "Mouser" "603-RT0805FRE075R1L"
 			(at 261.62 50.8 0)
 			(effects
@@
 			)
 		)
-		(property "TME" "AC0603FR-075R1L"
+		(property "TME" "CRCW08055R10FKTABC"
 			(at 261.62 50.8 0)
 			(effects
@@
 			)
 		)
-		(property "LCSC" "C227988"
+		(property "LCSC" "C364355"
 			(at 261.62 50.8 0)
 			(effects
@@
 			)
 		)
-		(property "DigiKey" "YAG5344CT-ND"
+		(property "DigiKey" "13-RT0805FRE075R1LCT-ND"
 			(at 254 50.8 0)
 			(effects
@@
 			)
 		)
-		(property "Mouser" " 603-AC0603FR-075R1L"
+		(property "Mouser" "603-RT0805FRE075R1L"
 			(at 254 50.8 0)
 			(effects
@@
 			)
 		)
-		(property "TME" "AC0603FR-075R1L"
+		(property "TME" "CRCW08055R10FKTABC"
 			(at 254 50.8 0)
 			(effects
@@
 			)
 		)
-		(property "MF" ""
-			(at 254 50.8 0)
-			(effects
-				(font
-					(size 1.27 1.27)
-				)
-				(hide yes)
-			)
-		)
-		(property "LCSC" "C227988"
+		(property "LCSC" "C364355"
 			(at 254 50.8 0)
 			(effects
