File: Experimental/KiCad/TFT DSI module/BB3plus DSI TFT display.kicad_pcb (KiCad board)
At the start: 2 copper layers, 136 x 92 mm, 50 parts, among them IC1 AZ1117CH2-3.3TRG1, IC2 TCA9554APWR, IC3 TPS61169DCKR, SW1 B3FS-4052P, SW2 B3FS-4052P, SW3 B3FS-4052P, SW4 B3FS-4052P, X1 5051102091, X2 505110-4091, X3 F3311A7H121010E200

Commit message: Enclosure front and rear panel update, projects location reorganized
Parts:
- X1: value 5051102091 -> 5051102291
Changed lines of the file:
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@@
 			)
 		)
-		(property "Value" "5051102091"
+		(property "Value" "5051102291"
 			(at 0 0 0)
 			(unlocked yes)
@@
 			(keep_text_aligned yes)
 		)
-		(gr_text "67,4 mm"
+		(gr_text "2653,5 mils"
 			(at 102.55 93.3 90)
 			(layer "Dwgs.User")
@@
 			(keep_text_aligned yes)
 		)
-		(gr_text "75,8 mm"
+		(gr_text "2983,9 mils"
 			(at 96.12 95.495 90)
 			(layer "Dwgs.User")
@@
 			(keep_text_aligned yes)
 		)
-		(gr_text "116,0 mm"
+		(gr_text "4566,9 mils"
 			(at 153 143.15 0)
 			(layer "User.1")
@@
 			(keep_text_aligned yes)
 		)
-		(gr_text "84,0 mm"
+		(gr_text "3307,1 mils"
 			(at 223.95 95.5 90)
 			(layer "User.1")
@@
 			(keep_text_aligned yes)
 		)
-		(gr_text "4,9 mm"
+		(gr_text "192,9 mils"
 			(at 208.55 138.05 0)
 			(layer "User.1")
@@
 			(keep_text_aligned yes)
 		)
-		(gr_text "4,0 mm"
+		(gr_text "157,5 mils"
 			(at 223.95 139.5 90)
 			(layer "User.1")
@@
 			(keep_text_aligned yes)
 		)
-		(gr_text "4,0 mm"
+		(gr_text "157,5 mils"
 			(at 223.95 51.500002 90)
 			(layer "User.1")
@@
 			(keep_text_aligned yes)
 		)
-		(gr_text "92,0 mm"
+		(gr_text "3622,0 mils"
 			(at 226.760496 95.5 90)
 			(layer "User.1")
@@
 			(keep_text_aligned yes)
 		)
-		(gr_text "10,0 mm"
+		(gr_text "393,7 mils"
 			(at 90.000001 143.15 0)
 			(layer "User.1")
@@
 			(keep_text_aligned yes)
 		)
-		(gr_text "44,0 mm"
+		(gr_text "1732,3 mils"
 			(at 132.799887 111.4 90)
 			(layer "User.1")
@@
 			(keep_text_aligned yes)
 		)
-		(gr_text "30,4 mm"
+		(gr_text "1195,1 mils"
 			(at 177.69 118.2225 90)
 			(layer "User.1")
@@
 			(keep_text_aligned yes)
 		)
-		(gr_text "34,0 mm"
+		(gr_text "1339,0 mils"
 			(at 204.005 106.41 0)
 			(layer "User.1")
@@
 			(keep_text_aligned yes)
 		)
-		(gr_text "84,0 mm"
+		(gr_text "3307,1 mils"
 			(at 179 92.66 0)
 			(layer "User.1")
@@
 			(keep_text_aligned yes)
 		)
-		(gr_text "10,0 mm"
+		(gr_text "393,7 mils"
 			(at 216 143.15 0)
 			(layer "User.1")
@@
 			(keep_text_aligned yes)
 		)
-		(gr_text "136,0 mm"
+		(gr_text "5354,3 mils"
 			(at 153 145.25 0)
 			(layer "User.1")
