File: KiCad/Enclosure/BB3plus enclosure front panel.kicad_pcb (KiCad board)
At the start: 4 copper layers, 0 parts

Commit message: Enclosure front and rear panel update, projects location reorganized
Other:
- copper layers 4 -> 2
