File: KiCad/Enclosure/BB3plus enclosure rear panel.kicad_pcb (KiCad board)
At the start: 4 copper layers, 0 parts

Commit message: Enclosure front panel
Other:
- board text added: "90"
- board text added: "Countersink hole detail"

Commit message: Enclosure front and rear panel update, projects location reorganized
Other:
- copper layers 4 -> 2
