File: KiCad/Enclosure/BB3plus enclosure bottom plate.kicad_pcb (KiCad board)
At the start: 4 copper layers, 0 parts

Commit message: Enclosure front and rear panel update, projects location reorganized
Other:
- copper layers 4 -> 2
- board text added: "Bottom panel, top (inside) view"
- board text removed: "Bottom panel, top view"
Changed lines of the file:
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@@
 	(layers
 		(0 "F.Cu" signal)
-		(4 "In1.Cu" power)
-		(6 "In2.Cu" signal)
 		(2 "B.Cu" signal)
 		(9 "F.Adhes" user "F.Adhesive")
@@
 			)
 			(layer "dielectric 1"
-				(type "prepreg")
-				(thickness 0.21)
-				(material "FR4")
-				(epsilon_r 4.5)
-				(loss_tangent 0.02)
-			)
-			(layer "In1.Cu"
-				(type "copper")
-				(thickness 0.015)
-			)
-			(layer "dielectric 2"
 				(type "core")
-				(thickness 1.065)
-				(material "FR4")
-				(epsilon_r 4.5)
-				(loss_tangent 0.02)
-			)
-			(layer "In2.Cu"
-				(type "copper")
-				(thickness 0.015)
-			)
-			(layer "dielectric 3"
-				(type "prepreg")
-				(thickness 0.21)
+				(thickness 1.515)
 				(material "FR4")
 				(epsilon_r 4.5)
@@
 		(layer "User.4")
 	)
+	(gr_circle
+		(center 305.75 58.25)
+		(end 307.25 58.25)
+		(stroke
+			(width 0.1)
+			(type solid)
+		)
+		(fill no)
+		(layer "User.4")
+	)
 	(gr_line
 		(start 547.810251 -131.960264)
@@
 		(layer "User.4")
 	)
+	(gr_circle
+		(center 438.75 161.95)
+		(end 440.25 161.95)
+		(stroke
+			(width 0.1)
+			(type solid)
+		)
+		(fill no)
+		(layer "User.4")
+	)
 	(gr_line
 		(start 302.55 -43.102479)
@@
 		(stroke
 			(width 0.1)
-			(type solid)
+			(type dash)
 		)
 		(fill no)
@@
 		(layer "User.4")
 	)
+	(gr_circle
+		(center 531.75 58.25)
+		(end 533.25 58.25)
+		(stroke
+			(width 0.1)
+			(type solid)
+		)
+		(fill no)
+		(layer "User.4")
+	)
+	(gr_circle
+		(center 519.75 -42.75)
+		(end 521.25 -42.75)
+		(stroke
+			(width 0.1)
+			(type solid)
+		)
+		(fill no)
+		(layer "User.4")
+	)
 	(gr_line
 		(start 293.6 -152.5)
@@
 		(layer "User.4")
 	)
+	(gr_circle
+		(center 429.75 -44.95)
+		(end 431.25 -44.95)
+		(stroke
+			(width 0.1)
+			(type solid)
+		)
+		(fill no)
+		(layer "User.4")
+	)
 	(gr_line
 		(start 642.999423 -49.845715)
@@
 		(stroke
 			(width 0.1)
-			(type dash)
+			(type solid)
 		)
 		(layer "User.4")
@@
 		(stroke
 			(width 0.1)
-			(type solid)
+			(type dash)
 		)
 		(fill no)
@@
 		(layer "User.4")
 	)
+	(gr_circle
+		(center 305.75 161.95)
+		(end 307.25 161.95)
+		(stroke
+			(width 0.1)
+			(type solid)
+		)
+		(fill no)
+		(layer "User.4")
+	)
 	(gr_line
 		(start 547.746751 -134.119255)
@@
 		(layer "User.4")
 	)
+	(gr_circle
+		(center 531.75 161.95)
+		(end 533.25 161.95)
+		(stroke
+			(width 0.1)
+			(type solid)
+		)
+		(fill no)
+		(layer "User.4")
+	)
 	(gr_line
 		(start 643.12646 171.134009)
@@
 		(stroke
 			(width 0.1)
-			(type dash)
+			(type solid)
 		)
 		(layer "User.4")
@@
 		(layer "User.4")
 	)
+	(gr_circle
+		(center 305.75 -44.95)
+		(end 307.25 -44.95)
+		(stroke
+			(width 0.1)
+			(type solid)
+		)
+		(fill no)
+		(layer "User.4")
+	)
 	(gr_line
 		(start 643.189923 167.832013)
@@
 		)
 	)
-	(gr_text "Bottom panel, top view"
+	(gr_text "Bottom panel, top (inside) view"
 		(at 293.5 -67.25 0)
 		(layer "User.4")
@@
 			(thickness 0.1)
 			(arrow_length 1.27)
-			(text_position_mode 0)
+			(text_position_mode 2)
 			(arrow_direction outward)
 			(extension_height 0.58642)
@@
 		)
 		(gr_text "1,5"
-			(at 294.25 174.16 0)
+			(at 292.04 175.27 0)
 			(layer "User.3")
 			(effects
