File: KiCad/Enclosure/BB3plus enclosure top plate.kicad_pcb (KiCad board)
At the start: 4 copper layers, 0 parts

Commit message: Enclosure front panel
Other:
- board text added: "Countersunk hole detail"
- board text removed: "Countersink hole detail"

Commit message: #1, #3, #4
Other:
- board text added: "Front panel"
- board text added: "Rear panel"
