File: KiCad/Front masks/Bare front mask half width.kicad_pcb (KiCad board)
At the start: 2 copper layers, 17.2 x 111.5 mm, 3 parts

Commit message: #5, #6
Parts:
- REF** (x2): footprint PCM_EEZ_THT:Mounting_hole 2_4.4mm_via_NO_NET -> PCM_EEZ_THT:Mounting_hole 1.8_4.4mm_via_NO_NET
- moved G*** 0.91 mm to (148.6, 93.5)
