File: Experimental/KiCad/DIB2 USB adapter/DIB2 USB adapter.kicad_pcb (KiCad board)
At the start: 4 copper layers, 91.3 x 92.5 mm, 21 parts, among them X2 10018783-10101TLF, X3 USB1135-15-9-L-B_REVA1

Commit message: USB adapter wiring fixed
Connections:
- X3 pad 2: /DIB_USB_D+ -> /DIB_USB_D-
- X3 pad 3: /DIB_USB_D- -> /DIB_USB_D+
- X3 pad 5: /USB3_RX+ -> /USB3_RX-
- X3 pad 6: /USB3_RX- -> /USB3_RX+
Routing:
- net /USB3_TX-: track 96.7 -> 105.9 mm
- net /USB3_TX+: track 97.2 -> 106.0 mm
- net /DIB_USB_D+: track 99.6 -> 91.2 mm
- net /DIB_USB_D-: track 98.8 -> 91.4 mm
- net /USB3_RX+: track 98.0 -> 105.4 mm
- net /USB3_RX-: track 98.0 -> 105.4 mm
- net /DIB_SCLK: track 105.7 -> 108.3 mm
- net /DIB_MISO: track 110.9 -> 113.2 mm, vias 1 -> 2
- net +5V: track 93.6 -> 91.4 mm
- net /DIB_MOSI: track 107.6 -> 109.3 mm
- net /~{DIB_CSA}: track 114.7 -> 116.4 mm, vias 1 -> 2
- net GND: track 33.7 -> 33.0 mm
- net /DIB_IRQ: track 112.7 -> 113.4 mm
- net PE: track 111.7 -> 111.1 mm, vias 0 -> 1
- added copper zone on F.Cu, net +12V
Other:
- board text added: "EEZ DIB2 Adapter (06/2026 ${project_version})"
- board text removed: "EEZ DIB2 Adapter (03/2026 ${project_version})"
