File: KiCad/BB3plus mainboard/BB3plus mainboard.kicad_pcb (KiCad board)
At the start: 4 copper layers, 233 x 230.5 mm, 420 parts, among them IC1 SN74HCS02PWR, IC10 SN6505BDBVR, IC11 EMC2301-1-ACZL-TR, IC12 ISO6763FDWR, IC13 BD00FC0W, IC14 THVD1420DR, IC15 TPS7A2050PDBVR, IC16 TPS7A2033PDBVR, IC17 TPD4E001DRLR, IC18 TPD4E001DRLR, IC19 USB5807C/KD, IC2 M24C32-DFDW6TP, IC20 TPS62933ODRLR, IC21 PTN5150AHXMP, IC22 MIC2026A-1YM-TR, IC23 TPS2068E, IC24 TPD4E001DRLR, IC25 FUSB340TMX, IC26 TPS22948DCKR, IC27 TLE75008ESDXUMA1, IC3 SN74LVC1G74DCUR, IC4 SN74LVC1G57DCKR, IC5 STM32G071R8T6, IC6 TPS3851H18EDRBR, IC7 SN74LVC00, IC8 TPS62933ODRLR, IC9 LM64460CPPQRYFRQ1, K1 AZ943-1CH-12DE, K2 AZ943-1CH-12DE, K3 RT424012, K4 RT424012, K5 RT424012, K6 RT424012, K7 RT424012, Q1 2N7002, Q2 2N7002, Q3 2N7002, Q4 MMBT5401, Q5 2N7002, Q6 DMP3013SFV-7, Q7 2N7002, Q8 2N7002, SW1 WBL2UOAGQR05CLR, SW2 PEC16-2215F-S0024, X1 DF40HC(3.0)-100DS-0.4V(51), X10 B3P-VH-FB-B, X11 B3P-VH-FB-B, X12 22-27-2031, X13 TBP03R1-350-10BE, X14 0862-1J1T-43-F, X15 USB4056-03-A, X16 SS-53000-002, X17 505110-2291, X18 505110-2291, X19 1001878410201TLF, X2 DF40HC(3.0)-100DS-0.4V(51), X20 1001878410201TLF, X21 1001878410201TLF, X22 1001878410201TLF, X23 1001878410201TLF, X24 77313-802-20LF, X25 77313-802-20LF, X26 TBP03R1-350-10BE, X27 77313-802-20LF, X3 1-2199230-6, X5 571-0400, X6 GSP1.9101.1, X7 1-726388-2, X8 B3P-VH-FB-B, X9 B3P-VH-FB-B, Y1 FC-135 32.7680KA-K0, Y2 VXM7-9032-25M0000000

Commit message: #12
Parts:
- IC7: value SN74LVC00 -> SN74HCS02PWR
Connections:
- IC7 pad 1: /System MCU, Watchdog, EEPROM/RTC_OUT -> RTC_FAN
- IC7 pad 10: /System MCU, Watchdog, EEPROM/RTC_OUT -> RTC_CM5
- IC7 pad 11: AC_FREQ -> Net-(IC7D-4A)
- IC7 pad 13: Net-(IC7D-4A) -> AC_FREQ
- IC7 pad 3: RTC_FAN -> /System MCU, Watchdog, EEPROM/RTC_OUT
- IC7 pad 4: /System MCU, Watchdog, EEPROM/RTC_OUT -> RTC_M2
- IC7 pad 6: RTC_M2 -> /System MCU, Watchdog, EEPROM/RTC_OUT
- IC7 pad 8: RTC_CM5 -> /System MCU, Watchdog, EEPROM/RTC_OUT
Routing:
- net Net-(IC7D-4A): track 152.6 -> 154.4 mm
- net RTC_FAN: track 97.7 -> 96.2 mm
- net RTC_M2: track 34.8 -> 35.9 mm
- net AC_FREQ: track 130.6 -> 131.4 mm
- net RTC_CM5: track 97.2 -> 98.0 mm
