File: KiCad/BB3plus mainboard/cm5_socket.kicad_sch (KiCad schematic)
At the start: 21 parts, among them Q1 2N7002, X1 DF40HC(3.0)-100DS-0.4V(51), X2 DF40HC(3.0)-100DS-0.4V(51), X3 1-2199230-6

Commit message: #17
Connections:
- net ~{LED_PWR}: now reaches Q1.1 (G), X1.95 (LED_nPWR)
Changed lines of the file:
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@@
+		)
+	)
+	(label "~{LED_PWR}"
+		(at 101.6 147.32 0)
+		(effects
+			(font
+				(size 0.889 0.889)
+			)
+			(justify left bottom)
 		)
 	)

Commit message: #18
Connections:
- net ~{LED_PWR} renamed CM5_LED_PWR
Changed lines of the file:
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@@
 	)
 	(junction
+		(at 116.84 147.32)
+		(diameter 0)
+		(color 0 0 0 0)
+	)
+	(junction
 		(at 99.06 129.54)
 		(diameter 0)
@@
 	(wire
 		(pts
+			(xy 116.84 147.32) (xy 119.38 147.32)
+		)
+		(stroke
+			(width 0)
+			(type default)
+		)
+	)
+	(wire
+		(pts
 			(xy 220.98 43.18) (xy 236.22 43.18)
 		)
@@
 		)
 	)
-	(label "~{LED_PWR}"
-		(at 101.6 147.32 0)
-		(effects
-			(font
-				(size 0.889 0.889)
-			)
-			(justify left bottom)
-		)
-	)
 	(label "PCIe_nWAKE"
 		(at 127 30.48 0)
@@
 			)
 		)
+	)
+	(global_label "CM5_LED_PWR"
+		(shape output)
+		(at 119.38 147.32 0)
+		(fields_autoplaced yes)
+		(effects
+			(font
+				(size 0.889 0.889)
+			)
+			(justify left)
+		)
+		(property "Intersheetrefs" "${INTERSHEET_REFS}"
+			(at 130.3249 147.32 0)
+			(hide yes)
+			(show_name no)
+			(do_not_autoplace no)
+			(effects
+				(font
+					(size 1.27 1.27)
+				)
+				(justify left)
+			)
+		)

Commit message: #19
Connections:
- net DIN2: now also X1.97 (CAM_GPIO0); no longer X1.35 (ID_SC/GPIO1)
- net RS485_RX/DIN3: now also X1.35 (ID_SC/GPIO1); no longer X1.100 (CAM_GPIO1)
- net RS485_TX/DOUT3: now also X1.36 (ID_SD/GPIO0); no longer X1.97 (CAM_GPIO0)
- net RTC_CM5: now also X1.100 (CAM_GPIO1); no longer X1.36 (ID_SD/GPIO0)
Changed lines of the file:
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@@
 	(title_block
 		(title "${project_name}")
-		(date "2026-09-13")
+		(date "2026-09-17")
 		(rev "${project_version}")
 		(company "${project_creator}")
@@
 	(wire
 		(pts
-			(xy 93.98 71.12) (xy 101.6 71.12)
-		)
-		(stroke
-			(width 0)
-			(type default)
-		)
-	)
-	(wire
-		(pts
 			(xy 93.98 30.48) (xy 101.6 30.48)
 		)
@@
 	(wire
 		(pts
-			(xy 93.98 149.86) (xy 101.6 149.86)
-		)
-		(stroke
-			(width 0)
-			(type default)
-		)
-	)
-	(wire
-		(pts
 			(xy 195.58 78.74) (xy 200.66 78.74)
 		)
@@
 	(wire
 		(pts
+			(xy 93.98 71.12) (xy 101.6 71.12)
+		)
+		(stroke
+			(width 0)
+			(type default)
+		)
+	)
+	(wire
+		(pts
 			(xy 213.36 78.74) (xy 213.36 81.28)
 		)
@@
 	(wire
 		(pts
-			(xy 35.56 71.12) (xy 43.18 71.12)
+			(xy 22.86 114.3) (xy 25.4 114.3)
 		)
 		(stroke
@@
 	(wire
 		(pts
-			(xy 22.86 114.3) (xy 25.4 114.3)
+			(xy 93.98 68.58) (xy 96.52 68.58)
 		)
 		(stroke
@@
 	(wire
 		(pts
-			(xy 93.98 68.58) (xy 96.52 68.58)
+			(xy 195.58 71.12) (xy 200.66 71.12)
 		)
 		(stroke
@@
 	(wire
 		(pts
-			(xy 195.58 71.12) (xy 200.66 71.12)
+			(xy 40.64 149.86) (xy 40.64 157.48)
 		)
 		(stroke
@@
 	(wire
 		(pts
-			(xy 40.64 149.86) (xy 40.64 157.48)
+			(xy 134.62 137.16) (xy 139.7 137.16)
 		)
 		(stroke
@@
 	(wire
 		(pts
-			(xy 134.62 137.16) (xy 139.7 137.16)
+			(xy 220.98 30.48) (xy 236.22 30.48)
 		)
 		(stroke
@@
 	(wire
 		(pts
-			(xy 220.98 30.48) (xy 236.22 30.48)
+			(xy 25.4 111.76) (xy 25.4 114.3)
 		)
 		(stroke
@@
 	(wire
 		(pts
-			(xy 25.4 111.76) (xy 25.4 114.3)
+			(xy 35.56 71.12) (xy 43.18 71.12)
 		)
 		(stroke
@@
 	(wire
 		(pts
+			(xy 33.02 152.4) (xy 43.18 152.4)
+		)
+		(stroke
+			(width 0)
+			(type default)
+		)
+	)
+	(wire
+		(pts
 			(xy 220.98 40.64) (xy 236.22 40.64)
 		)
@@
 		)
 	)
-	(wire
-		(pts
-			(xy 33.02 152.4) (xy 43.18 152.4)
-		)
-		(stroke
-			(width 0)
-			(type default)
-		)
-	)
 	(polyline
 		(pts
@@
 		)
 	)
+	(wire
+		(pts
+			(xy 93.98 149.86) (xy 101.6 149.86)
+		)
+		(stroke
+			(width 0)
+			(type default)
+		)
+	)
 	(polyline
 		(pts
@@
 	(global_label "RTC_CM5"
 		(shape input)
-		(at 35.56 71.12 180)
+		(at 33.02 152.4 180)
 		(fields_autoplaced yes)
 		(effects
@@
 		)
 		(property "Intersheetrefs" "${INTERSHEET_REFS}"
-			(at 28.0441 71.12 0)
+			(at 25.5041 152.4 0)
 			(hide yes)
 			(show_name no)
@@
 	(global_label "RS485_TX{slash}DOUT3"
 		(shape output)
-		(at 101.6 149.86 0)
+		(at 35.56 71.12 180)
 		(fields_autoplaced yes)
 		(effects
@@
 				(size 0.889 0.889)
 			)
-			(justify left)
+			(justify right)
 		)
 		(property "Intersheetrefs" "${INTERSHEET_REFS}"
-			(at 114.9156 149.86 0)
+			(at 22.2444 71.12 0)
 			(hide yes)
 			(show_name no)
@@
 					(size 1.27 1.27)
 				)
-				(justify left)
+				(justify right)
 			)
 		)
@@
 	(global_label "DIN2"
 		(shape input)
-		(at 101.6 71.12 0)
+		(at 101.6 149.86 0)
 		(fields_autoplaced yes)
 		(effects
@@
 		)
 		(property "Intersheetrefs" "${INTERSHEET_REFS}"
-			(at 106.3219 71.12 0)
+			(at 106.3219 149.86 0)
 			(hide yes)
 			(show_name no)
@@
 	(global_label "RS485_RX{slash}DIN3"
 		(shape input)
-		(at 33.02 152.4 180)
+		(at 101.6 71.12 0)
 		(fields_autoplaced yes)
 		(effects
@@
 				(size 0.889 0.889)
 			)
-			(justify right)
+			(justify left)
 		)
 		(property "Intersheetrefs" "${INTERSHEET_REFS}"
-			(at 20.678 152.4 0)
+			(at 113.942 71.12 0)
 			(hide yes)
 			(show_name no)
@@
 					(size 1.27 1.27)
 				)
-				(justify right)
+				(justify left)
 			)
 		)

Commit message: BOM update
Parts:
- X3: value 1-2199230-6 -> SM3ZS067U410AMR1000; DigiKey A118046TR-ND -> 670-2693-1-ND; LCSC C4710843 -> C5078373; Mouser 571-1-2199230-6 -> 656-SM3ZS067U410AM10
Changed lines of the file:
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@@
 	(title_block
 		(title "${project_name}")
-		(date "2026-09-17")
+		(date "2026-09-19")
 		(rev "${project_version}")
 		(company "${project_creator}")
@@
 			)
 		)
-		(property "Value" "1-2199230-6"
+		(property "Value" "SM3ZS067U410AMR1000"
 			(at 243.84 107.9499 0)
 			(hide yes)
@@
 			)
 		)
-		(property "DigiKey" "A118046TR-ND"
+		(property "DigiKey" "670-2693-1-ND"
 			(at 241.3 111.76 0)
 			(hide yes)
@@
 			)
 		)
-		(property "Mouser" "571-1-2199230-6"
+		(property "Mouser" "656-SM3ZS067U410AM10"
 			(at 241.3 111.76 0)
 			(hide yes)
@@
 			)
 		)
-		(property "LCSC" "C4710843"
+		(property "LCSC" "C5078373"
 			(at 241.3 111.76 0)
 			(hide yes)
@@
 			)
 		)
-		(property "Value" "1-2199230-6"
+		(property "Value" "SM3ZS067U410AMR1000"
 			(at 238.76 99.695 0)
 			(show_name no)
@@
 			)
 		)
-		(property "DigiKey" "A118046TR-ND"
+		(property "DigiKey" "670-2693-1-ND"
 			(at 238.76 25.4 0)
 			(hide yes)
@@
 			)
 		)
-		(property "Mouser" "571-1-2199230-6"
+		(property "Mouser" "656-SM3ZS067U410AM10"
 			(at 238.76 25.4 0)
 			(hide yes)
@@
 			)
 		)
-		(property "LCSC" "C4710843"
+		(property "LCSC" "C5078373"
 			(at 238.76 25.4 0)
 			(hide yes)
