File: KiCad/BB3plus mainboard/cm5_socket.kicad_sch (KiCad schematic)
At the start: 21 parts, among them Q1 2N7002, X1 DF40HC(3.0)-100DS-0.4V(51), X2 DF40HC(3.0)-100DS-0.4V(51), X3 SM3ZS067U410AMR1000

Commit message: Rear USB & Ethernet updated
Parts:
- JP3: Label CM5_BOOT0 -> CM5_BOOT
Connections:
- net CM5_BOOT0 renamed CM5_BOOT
Changed lines of the file:
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@@
 		)
 	)
-	(global_label "CM5_BOOT0"
+	(global_label "CM5_BOOT"
 		(shape input)
 		(at 104.14 144.78 0)
@@
 		(in_bom no)
 		(on_board yes)
-		(in_pos_files yes)
+		(in_pos_files no)
 		(dnp no)
 		(property "Reference" "JP4"
@@
 			)
 		)
-		(property "Label" "CM5_BOOT0"
+		(property "Label" "CM5_BOOT"
 			(at 109.22 137.16 90)
 			(show_name no)
@@
 		(in_bom no)
 		(on_board yes)
-		(in_pos_files yes)
+		(in_pos_files no)
 		(dnp no)
 		(property "Reference" "JP5"
