File: KiCad/BB3plus mainboard/cm5_socket.kicad_sch (KiCad schematic)
At the start: 21 parts, among them Q1 2N7002, X1 DF40HC(3.0)-100DS-0.4V(51), X2 DF40HC(3.0)-100DS-0.4V(51), X3 SM3ZS067U410AMR1000

Commit message: BOM and DIB2 specification updated
Parts:
- C1: DigiKey 490-5523-1-ND -> 490-GRM21BR61E106MA73KCT-ND; Mouser 81-GRM21BR61E106KA3L -> 81-GRM21BR61C106KE5K; TME GRM21BR61E106KA73L -> CL21A106KAYNNNE
- LED1: DigiKey 160-1414-2-ND -> 160-1414-1-ND
- R3, R4, R7: DigiKey 311-330HRCT-ND -> 311-330LMCT-ND
- R5, R6: DigiKey 1712-CRGH0603F10KCT-ND -> 13-RC0603FR-1310KLCT-ND; Mouser 756-WCR0603-10KFI -> 603-RC0603FR-1310KL; TME SMD0603-10K-1% -> RC0603FR-0710K
- X1, X2: DigiKey 26-DF40HC(3.0)-100DS-0.4V(51)CT-ND -> H124602CT-ND; Mouser 798-DF40HC30100DS451 -> 798-DF40HC30100DS458; TME - -> DF40HC30100DS04V58
Changed lines of the file:
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@@
 	(title_block
 		(title "${project_name}")
-		(date "2026-10-25")
+		(date "2026-10-31")
 		(rev "${project_version}")
 		(company "${project_creator}")
@@
 			)
 		)
-		(property "DigiKey" "311-330HRCT-ND"
+		(property "DigiKey" "311-330LMCT-ND"
 			(at 116.84 38.1 0)
 			(hide yes)
@@
 			)
 		)
-		(property "DigiKey" "1712-CRGH0603F10KCT-ND"
+		(property "DigiKey" "13-RC0603FR-1310KLCT-ND"
 			(at 213.36 73.66 0)
 			(hide yes)
@@
 			)
 		)
-		(property "Mouser" "756-WCR0603-10KFI"
+		(property "Mouser" "603-RC0603FR-1310KL"
 			(at 213.36 73.66 0)
 			(hide yes)
@@
 			)
 		)
-		(property "TME" "SMD0603-10K-1%"
+		(property "TME" "RC0603FR-0710K"
 			(at 213.36 73.66 0)
 			(hide yes)
@@
 			)
 		)
-		(property "DigiKey" "490-5523-1-ND"
+		(property "DigiKey" "490-GRM21BR61E106MA73KCT-ND"
 			(at 231.14 93.98 0)
 			(hide yes)
@@
 			)
 		)
-		(property "Mouser" "81-GRM21BR61E106KA3L"
+		(property "Mouser" "81-GRM21BR61C106KE5K"
 			(at 231.14 93.98 0)
 			(hide yes)
@@
 			)
 		)
-		(property "TME" "GRM21BR61E106KA73L"
+		(property "TME" "CL21A106KAYNNNE"
 			(at 231.14 93.98 0)
 			(hide yes)
@@
 			)
 		)
-		(property "DigiKey" "26-DF40HC(3.0)-100DS-0.4V(51)CT-ND"
+		(property "DigiKey" "H124602CT-ND"
 			(at 144.78 160.02 0)
 			(hide yes)
@@
 			)
 		)
-		(property "Mouser" "798-DF40HC30100DS451 "
+		(property "Mouser" "798-DF40HC30100DS458"
 			(at 144.78 162.56 0)
 			(hide yes)
@@
 			)
 		)
-		(property "TME" "-"
+		(property "TME" "DF40HC30100DS04V58"
 			(at 144.78 165.1 0)
 			(hide yes)
@@
 			)
 		)
-		(property "DigiKey" "160-1414-2-ND"
+		(property "DigiKey" "160-1414-1-ND"
 			(at 116.84 55.88 0)
 			(hide yes)
@@
 			)
 		)
-		(property "DigiKey" "311-330HRCT-ND"
+		(property "DigiKey" "311-330LMCT-ND"
 			(at 127 167.64 0)
 			(hide yes)
@@
 			)
 		)
-		(property "DigiKey" "311-330HRCT-ND"
+		(property "DigiKey" "311-330LMCT-ND"
 			(at 269.24 63.5 0)
 			(hide yes)
@@
 			)
 		)
-		(property "DigiKey" "1712-CRGH0603F10KCT-ND"
+		(property "DigiKey" "13-RC0603FR-1310KLCT-ND"
 			(at 228.6 22.86 0)
 			(hide yes)
@@
 			)
 		)
-		(property "Mouser" "756-WCR0603-10KFI"
+		(property "Mouser" "603-RC0603FR-1310KL"
 			(at 228.6 22.86 0)
 			(hide yes)
@@
 			)
 		)
-		(property "TME" "SMD0603-10K-1%"
+		(property "TME" "RC0603FR-0710K"
 			(at 228.6 22.86 0)
 			(hide yes)
@@
 			)
 		)
-		(property "DigiKey" "26-DF40HC(3.0)-100DS-0.4V(51)CT-ND"
+		(property "DigiKey" "H124602CT-ND"
 			(at 45.72 160.02 0)
 			(hide yes)
@@
 			)
 		)
-		(property "Mouser" "798-DF40HC30100DS451 "
+		(property "Mouser" "798-DF40HC30100DS458"
 			(at 45.72 162.56 0)
 			(hide yes)
@@
 			)
 		)
-		(property "TME" "-"
+		(property "TME" "DF40HC30100DS04V58"
 			(at 45.72 165.1 0)
 			(hide yes)
