File: KiCad/BB3plus mainboard/power_coupling.kicad_sch (KiCad schematic)
At the start: 16 parts, among them IC28 TLE75008ESDXUMA1, K3 RT424012, K4 RT424012, K5 RT424012, K6 RT424012, K7 RT424012, X24 77313-802-20LF, X25 77313-802-20LF, X26 TBP03R1-350-10BE, X27 77313-802-20LF

Commit message: #17
Parts:
- renumbered C135 to C136, C136 to C137, C137 to C138, C138 to C139, D17 to D19, R97 to R96
Changed lines of the file:
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@@
 		(in_pos_files yes)
 		(dnp no)
-		(property "Reference" "C135"
+		(property "Reference" "C136"
 			(at 30.48 78.105 90)
 			(show_name no)
@@
 			(project "BB3plus mainboard"
 				(path "/1df84e4f-233a-4f72-9418-c0020706bb76/bb7e7620-5970-4f17-83aa-0b2c666475d0"
-					(reference "C135")
+					(reference "C136")
 					(unit 1)
 				)
@@
 		(in_pos_files yes)
 		(dnp no)
-		(property "Reference" "#+3V054"
+		(property "Reference" "#+3V053"
 			(at 76.2 106.68 0)
 			(hide yes)
@@
 			(project "BB3plus mainboard"
 				(path "/1df84e4f-233a-4f72-9418-c0020706bb76/bb7e7620-5970-4f17-83aa-0b2c666475d0"
-					(reference "#+3V054")
+					(reference "#+3V053")
 					(unit 1)
 				)
@@
 		(in_pos_files yes)
 		(dnp no)
-		(property "Reference" "C138"
+		(property "Reference" "C139"
 			(at 200.025 142.24 0)
 			(show_name no)
@@
 			(project "BB3plus mainboard"
 				(path "/1df84e4f-233a-4f72-9418-c0020706bb76/bb7e7620-5970-4f17-83aa-0b2c666475d0"
-					(reference "C138")
+					(reference "C139")
 					(unit 1)
 				)
@@
 		(in_pos_files yes)
 		(dnp no)
-		(property "Reference" "C137"
+		(property "Reference" "C138"
 			(at 200.025 129.54 0)
 			(show_name no)
@@
 			(project "BB3plus mainboard"
 				(path "/1df84e4f-233a-4f72-9418-c0020706bb76/bb7e7620-5970-4f17-83aa-0b2c666475d0"
-					(reference "C137")
+					(reference "C138")
 					(unit 1)
 				)
@@
 		(in_pos_files yes)
 		(dnp no)
-		(property "Reference" "R97"
+		(property "Reference" "R96"
 			(at 71.12 113.665 0)
 			(show_name no)
@@
 			(project "BB3plus mainboard"
 				(path "/1df84e4f-233a-4f72-9418-c0020706bb76/bb7e7620-5970-4f17-83aa-0b2c666475d0"
-					(reference "R97")
+					(reference "R96")
 					(unit 1)
 				)
@@
 		(in_pos_files yes)
 		(dnp no)
-		(property "Reference" "#+3V053"
+		(property "Reference" "#+3V052"
 			(at 35.56 73.66 0)
 			(hide yes)
@@
 			(project "BB3plus mainboard"
 				(path "/1df84e4f-233a-4f72-9418-c0020706bb76/bb7e7620-5970-4f17-83aa-0b2c666475d0"
-					(reference "#+3V053")
+					(reference "#+3V052")
 					(unit 1)
 				)
@@
 		(in_pos_files yes)
 		(dnp no)
-		(property "Reference" "C136"
+		(property "Reference" "C137"
 			(at 66.04 78.105 90)
 			(show_name no)
@@
 			(project "BB3plus mainboard"
 				(path "/1df84e4f-233a-4f72-9418-c0020706bb76/bb7e7620-5970-4f17-83aa-0b2c666475d0"
-					(reference "C136")
+					(reference "C137")
 					(unit 1)
 				)
@@
 		(in_pos_files yes)
 		(dnp no)
-		(property "Reference" "D17"
+		(property "Reference" "D19"
 			(at 68.58 117.475 0)
 			(show_name no)
@@
 			(project "BB3plus mainboard"
 				(path "/1df84e4f-233a-4f72-9418-c0020706bb76/bb7e7620-5970-4f17-83aa-0b2c666475d0"
-					(reference "D17")
+					(reference "D19")
 					(unit 1)
 				)

Commit message: ZD4 added, PCB layout for AC lines improved
Parts:
- added ZD4: SMF16CA, PCM_EEZ_SMD:SODFL3718X130N, symbol PCM_EEZ_discretes:DIODE_TVS
- renumbered D19 to D18
Connections:
- net +12V: now also ZD4.C
- net GND: now also ZD4.A
Changed lines of the file:
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@@
 	)
 	(junction
+		(at 60.96 71.12)
+		(diameter 0)
+		(color 0 0 0 0)
+	)
+	(junction
 		(at 276.86 78.74)
 		(diameter 0)
@@
 	)
 	(junction
+		(at 71.12 78.74)
+		(diameter 0)
+		(color 0 0 0 0)
+	)
+	(junction
 		(at 137.16 73.66)
 		(diameter 0)
@@
 	(wire
 		(pts
-			(xy 60.96 76.2) (xy 60.96 78.74)
+			(xy 60.96 68.58) (xy 60.96 71.12)
 		)
 		(stroke
@@
 	(wire
 		(pts
+			(xy 68.58 71.12) (xy 71.12 71.12)
+		)
+		(stroke
+			(width 0)
+			(type default)
+		)
+	)
+	(wire
+		(pts
 			(xy 208.28 149.86) (xy 220.98 149.86)
 		)
@@
 	(wire
 		(pts
+			(xy 60.96 71.12) (xy 60.96 78.74)
+		)
+		(stroke
+			(width 0)
+			(type default)
+		)
+	)
+	(wire
+		(pts
 			(xy 106.68 144.78) (xy 119.38 144.78)
 		)
@@
 	(wire
 		(pts
+			(xy 71.12 71.12) (xy 71.12 78.74)
+		)
+		(stroke
+			(width 0)
+			(type default)
+		)
+	)
+	(wire
+		(pts
 			(xy 172.72 30.48) (xy 180.34 30.48)
 		)
@@
 	)
 	(symbol
+		(lib_id "PCM_EEZ_discretes:DIODE_TVS")
+		(at 66.04 71.12 0)
+		(mirror y)
+		(unit 1)
+		(body_style 1)
+		(exclude_from_sim no)
+		(in_bom yes)
+		(on_board yes)
+		(in_pos_files yes)
+		(dnp no)
+		(property "Reference" "ZD4"
+			(at 64.77 68.58 0)
+			(show_name no)
+			(do_not_autoplace no)
+			(effects
+				(font
+					(size 1.27 1.27)
+				)
+				(justify bottom)
+			)
+		)
+		(property "Value" "SMF16CA"
+			(at 60.96 74.93 0)
+			(show_name no)
+			(do_not_autoplace no)
+			(effects
+				(font
+					(size 1.27 1.27)
+				)
+				(justify right bottom)
+			)
+		)
+		(property "Footprint" "PCM_EEZ_SMD:SODFL3718X130N"
+			(at 66.675 74.295 0)
+			(hide yes)
+			(show_name no)
+			(do_not_autoplace no)
+			(effects
+				(font
+					(size 1.27 1.27)
+				)
+			)
+		)
+		(property "Datasheet" ""
+			(at 66.04 71.12 0)
+			(hide yes)
+			(show_name no)
+			(do_not_autoplace no)
+			(effects
+				(font
+					(size 1.27 1.27)
+				)
+			)
+		)
+		(property "Description" ""
+			(at 66.04 71.12 0)
+			(hide yes)
+			(show_name no)
+			(do_not_autoplace no)
+			(effects
+				(font
+					(size 1.27 1.27)
+				)
+			)
+		)
+		(property "DigiKey" "4878-SMF16CADKR-ND"
+			(at 66.04 71.12 0)
+			(hide yes)
+			(show_name no)
+			(do_not_autoplace no)
+			(effects
+				(font
+					(size 1.27 1.27)
+				)
+			)
+		)
+		(property "Mouser" "637-SMF16CA"
+			(at 66.04 71.12 0)
+			(hide yes)
+			(show_name no)
+			(do_not_autoplace no)
+			(effects
+				(font
+					(size 1.27 1.27)
+				)
+			)
+		)
+		(property "TME" "SMF16CA-DIO"
+			(at 66.04 71.12 0)
+			(hide yes)
+			(show_name no)
+			(do_not_autoplace no)
+			(effects
+				(font
+					(size 1.27 1.27)
+				)
+			)
+		)
+		(property "LCSC" "C1851354"
+			(at 66.04 71.12 0)
+			(hide yes)
+			(show_name no)
+			(do_not_autoplace no)
+			(effects
+				(font
+					(size 0.889 0.889)
+				)
+			)
+		)
+		(pin "A"
+		)
+		(pin "C"
+		)
+		(instances
+			(project "BB3plus mainboard"
+				(path "/1df84e4f-233a-4f72-9418-c0020706bb76/bb7e7620-5970-4f17-83aa-0b2c666475d0"
+					(reference "ZD4")
+					(unit 1)
+				)
+			)
+		)
+	)
+	(symbol
 		(lib_id "PCM_EEZ_connectors:DIB 2.0 Power connector (backplane)")
 		(at 193.04 63.5 0)
@@
 		(in_pos_files yes)
 		(dnp no)
-		(property "Reference" "#SUPPLY0106"
+		(property "Reference" "#SUPPLY0105"
 			(at 60.96 124.46 0)
 			(hide yes)
@@
 			(project "BB3plus mainboard"
 				(path "/1df84e4f-233a-4f72-9418-c0020706bb76/bb7e7620-5970-4f17-83aa-0b2c666475d0"
-					(reference "#SUPPLY0106")
+					(reference "#SUPPLY0105")
 					(unit 1)
 				)
@@
 		(in_pos_files yes)
 		(dnp no)
-		(property "Reference" "#SUPPLY0104"
+		(property "Reference" "#SUPPLY0103"
 			(at 35.56 109.22 0)
 			(hide yes)
@@
 			(project "BB3plus mainboard"
 				(path "/1df84e4f-233a-4f72-9418-c0020706bb76/bb7e7620-5970-4f17-83aa-0b2c666475d0"
-					(reference "#SUPPLY0104")
+					(reference "#SUPPLY0103")
 					(unit 1)
 				)
@@
 		(in_pos_files yes)
 		(dnp no)
-		(property "Reference" "#SUPPLY0108"
+		(property "Reference" "#SUPPLY0107"
 			(at 137.16 144.78 0)
 			(hide yes)
@@
 			(project "BB3plus mainboard"
 				(path "/1df84e4f-233a-4f72-9418-c0020706bb76/bb7e7620-5970-4f17-83aa-0b2c666475d0"
-					(reference "#SUPPLY0108")
+					(reference "#SUPPLY0107")
 					(unit 1)
 				)
@@
 	(symbol
 		(lib_id "PCM_EEZ_symbols:+12V")
-		(at 60.96 73.66 0)
+		(at 60.96 66.04 0)
 		(unit 1)
 		(body_style 1)
@@
 		(in_pos_files yes)
 		(dnp no)
-		(property "Reference" "#SUPPLY0105"
-			(at 60.96 73.66 0)
+		(property "Reference" "#SUPPLY0104"
+			(at 60.96 66.04 0)
 			(hide yes)
 			(show_name no)
@@
 		)
 		(property "Value" "+12V"
-			(at 60.96 73.025 0)
+			(at 60.96 65.405 0)
 			(show_name no)
 			(do_not_autoplace no)
@@
 		)
 		(property "Footprint" ""
-			(at 60.96 73.66 0)
+			(at 60.96 66.04 0)
 			(hide yes)
 			(show_name no)
@@
 		)
 		(property "Datasheet" ""
-			(at 60.96 73.66 0)
+			(at 60.96 66.04 0)
 			(hide yes)
 			(show_name no)
@@
 		)
 		(property "Description" ""
-			(at 60.96 73.66 0)
+			(at 60.96 66.04 0)
 			(hide yes)
 			(show_name no)
@@
 			(project "BB3plus mainboard"
 				(path "/1df84e4f-233a-4f72-9418-c0020706bb76/bb7e7620-5970-4f17-83aa-0b2c666475d0"
-					(reference "#SUPPLY0105")
+					(reference "#SUPPLY0104")
 					(unit 1)
 				)
@@
 		(in_pos_files yes)
 		(dnp no)
-		(property "Reference" "#SUPPLY0103"
+		(property "Reference" "#SUPPLY0102"
 			(at 25.4 83.82 0)
 			(hide yes)
@@
 			(project "BB3plus mainboard"
 				(path "/1df84e4f-233a-4f72-9418-c0020706bb76/bb7e7620-5970-4f17-83aa-0b2c666475d0"
-					(reference "#SUPPLY0103")
+					(reference "#SUPPLY0102")
 					(unit 1)
 				)
@@
 		(in_pos_files yes)
 		(dnp no)
-		(property "Reference" "#SUPPLY0107"
+		(property "Reference" "#SUPPLY0106"
 			(at 71.12 83.82 0)
 			(hide yes)
@@
 			(project "BB3plus mainboard"
 				(path "/1df84e4f-233a-4f72-9418-c0020706bb76/bb7e7620-5970-4f17-83aa-0b2c666475d0"
-					(reference "#SUPPLY0107")
+					(reference "#SUPPLY0106")
 					(unit 1)
 				)
@@
 		(in_pos_files yes)
 		(dnp no)
-		(property "Reference" "D19"
+		(property "Reference" "D18"
 			(at 68.58 117.475 0)
 			(show_name no)
@@
 			(project "BB3plus mainboard"
 				(path "/1df84e4f-233a-4f72-9418-c0020706bb76/bb7e7620-5970-4f17-83aa-0b2c666475d0"
-					(reference "D19")
+					(reference "D18")
 					(unit 1)
 				)

Commit message: CM5_BOOT0 control modified
Parts:
- renumbered D18 to D19, R96 to R97
Changed lines of the file:
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@@
 		(in_pos_files yes)
 		(dnp no)
-		(property "Reference" "R96"
+		(property "Reference" "R97"
 			(at 71.12 113.665 0)
 			(show_name no)
@@
 			(project "BB3plus mainboard"
 				(path "/1df84e4f-233a-4f72-9418-c0020706bb76/bb7e7620-5970-4f17-83aa-0b2c666475d0"
-					(reference "R96")
+					(reference "R97")
 					(unit 1)
 				)
@@
 		(in_pos_files yes)
 		(dnp no)
-		(property "Reference" "D18"
+		(property "Reference" "D19"
 			(at 68.58 117.475 0)
 			(show_name no)
@@
 			(project "BB3plus mainboard"
 				(path "/1df84e4f-233a-4f72-9418-c0020706bb76/bb7e7620-5970-4f17-83aa-0b2c666475d0"
-					(reference "D18")
+					(reference "D19")
 					(unit 1)
 				)

Commit message: #21
Parts:
- renumbered C136 to C133, C137 to C134, C138 to C135, C139 to C136, D19 to D17, IC28 to IC25, R97 to R95

Commit message: #22
Parts:
- renumbered C133 to C138, C134 to C139, C135 to C140, C136 to C141, IC25 to IC28, R95 to R96
Changed lines of the file:
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@@
 	(title_block
 		(title "${project_name}")
-		(date "2026-10-06")
+		(date "2026-10-08")
 		(rev "${project_version}")
 		(company "${project_creator}")
@@
 		(in_pos_files yes)
 		(dnp no)
-		(property "Reference" "C133"
+		(property "Reference" "C138"
 			(at 30.48 78.105 90)
 			(show_name no)
@@
 			(project "BB3plus mainboard"
 				(path "/1df84e4f-233a-4f72-9418-c0020706bb76/bb7e7620-5970-4f17-83aa-0b2c666475d0"
-					(reference "C133")
+					(reference "C138")
 					(unit 1)
 				)
@@
 		(in_pos_files yes)
 		(dnp no)
-		(property "Reference" "#+3V053"
+		(property "Reference" "#+3V052"
 			(at 76.2 106.68 0)
 			(hide yes)
@@
 			(project "BB3plus mainboard"
 				(path "/1df84e4f-233a-4f72-9418-c0020706bb76/bb7e7620-5970-4f17-83aa-0b2c666475d0"
-					(reference "#+3V053")
+					(reference "#+3V052")
 					(unit 1)
 				)
@@
 		(in_pos_files yes)
 		(dnp no)
-		(property "Reference" "#SUPPLY0107"
+		(property "Reference" "#SUPPLY0114"
 			(at 60.96 124.46 0)
 			(hide yes)
@@
 			(project "BB3plus mainboard"
 				(path "/1df84e4f-233a-4f72-9418-c0020706bb76/bb7e7620-5970-4f17-83aa-0b2c666475d0"
-					(reference "#SUPPLY0107")
+					(reference "#SUPPLY0114")
 					(unit 1)
 				)
@@
 		(in_pos_files yes)
 		(dnp no)
-		(property "Reference" "C136"
+		(property "Reference" "C141"
 			(at 200.025 142.24 0)
 			(show_name no)
@@
 			(project "BB3plus mainboard"
 				(path "/1df84e4f-233a-4f72-9418-c0020706bb76/bb7e7620-5970-4f17-83aa-0b2c666475d0"
-					(reference "C136")
+					(reference "C141")
 					(unit 1)
 				)
@@
 		(in_pos_files yes)
 		(dnp no)
-		(property "Reference" "#SUPPLY0105"
+		(property "Reference" "#SUPPLY0112"
 			(at 35.56 109.22 0)
 			(hide yes)
@@
 			(project "BB3plus mainboard"
 				(path "/1df84e4f-233a-4f72-9418-c0020706bb76/bb7e7620-5970-4f17-83aa-0b2c666475d0"
-					(reference "#SUPPLY0105")
+					(reference "#SUPPLY0112")
 					(unit 1)
 				)
@@
 		(in_pos_files yes)
 		(dnp no)
-		(property "Reference" "#SUPPLY0109"
+		(property "Reference" "#SUPPLY0116"
 			(at 137.16 144.78 0)
 			(hide yes)
@@
 			(project "BB3plus mainboard"
 				(path "/1df84e4f-233a-4f72-9418-c0020706bb76/bb7e7620-5970-4f17-83aa-0b2c666475d0"
-					(reference "#SUPPLY0109")
+					(reference "#SUPPLY0116")
 					(unit 1)
 				)
@@
 		(in_pos_files yes)
 		(dnp no)
-		(property "Reference" "#SUPPLY0106"
+		(property "Reference" "#SUPPLY0113"
 			(at 60.96 66.04 0)
 			(hide yes)
@@
 			(project "BB3plus mainboard"
 				(path "/1df84e4f-233a-4f72-9418-c0020706bb76/bb7e7620-5970-4f17-83aa-0b2c666475d0"
-					(reference "#SUPPLY0106")
+					(reference "#SUPPLY0113")
 					(unit 1)
 				)
@@
 		(in_pos_files yes)
 		(dnp no)
-		(property "Reference" "#SUPPLY0104"
+		(property "Reference" "#SUPPLY0111"
 			(at 25.4 83.82 0)
 			(hide yes)
@@
 			(project "BB3plus mainboard"
 				(path "/1df84e4f-233a-4f72-9418-c0020706bb76/bb7e7620-5970-4f17-83aa-0b2c666475d0"
-					(reference "#SUPPLY0104")
+					(reference "#SUPPLY0111")
 					(unit 1)
 				)
@@
 		(in_pos_files yes)
 		(dnp no)
-		(property "Reference" "#SUPPLY0108"
+		(property "Reference" "#SUPPLY0115"
 			(at 71.12 83.82 0)
 			(hide yes)
@@
 			(project "BB3plus mainboard"
 				(path "/1df84e4f-233a-4f72-9418-c0020706bb76/bb7e7620-5970-4f17-83aa-0b2c666475d0"
-					(reference "#SUPPLY0108")
+					(reference "#SUPPLY0115")
 					(unit 1)
 				)
@@
 		(in_pos_files yes)
 		(dnp no)
-		(property "Reference" "C135"
+		(property "Reference" "C140"
 			(at 200.025 129.54 0)
 			(show_name no)
@@
 			(project "BB3plus mainboard"
 				(path "/1df84e4f-233a-4f72-9418-c0020706bb76/bb7e7620-5970-4f17-83aa-0b2c666475d0"
-					(reference "C135")
+					(reference "C140")
 					(unit 1)
 				)
@@
 		(in_pos_files yes)
 		(dnp no)
-		(property "Reference" "R95"
+		(property "Reference" "R96"
 			(at 71.12 113.665 0)
 			(show_name no)
@@
 			(project "BB3plus mainboard"
 				(path "/1df84e4f-233a-4f72-9418-c0020706bb76/bb7e7620-5970-4f17-83aa-0b2c666475d0"
-					(reference "R95")
+					(reference "R96")
 					(unit 1)
 				)
@@
 		(in_pos_files yes)
 		(dnp no)
-		(property "Reference" "#+3V052"
+		(property "Reference" "#+3V051"
 			(at 35.56 73.66 0)
 			(hide yes)
@@
 			(project "BB3plus mainboard"
 				(path "/1df84e4f-233a-4f72-9418-c0020706bb76/bb7e7620-5970-4f17-83aa-0b2c666475d0"
-					(reference "#+3V052")
+					(reference "#+3V051")
 					(unit 1)
 				)
@@
 		(dnp no)
 		(fields_autoplaced yes)
-		(property "Reference" "IC25"
+		(property "Reference" "IC28"
 			(at 40.64 80.645 0)
 			(show_name no)
@@
 			(project "BB3plus mainboard"
 				(path "/1df84e4f-233a-4f72-9418-c0020706bb76/bb7e7620-5970-4f17-83aa-0b2c666475d0"
-					(reference "IC25")
+					(reference "IC28")
 					(unit 1)
 				)
@@
 		(in_pos_files yes)
 		(dnp no)
-		(property "Reference" "C134"
+		(property "Reference" "C139"
 			(at 66.04 78.105 90)
 			(show_name no)
@@
 			(project "BB3plus mainboard"
 				(path "/1df84e4f-233a-4f72-9418-c0020706bb76/bb7e7620-5970-4f17-83aa-0b2c666475d0"
-					(reference "C134")
+					(reference "C139")
 					(unit 1)
 				)
