File: KiCad/BB3plus mainboard/usb3_hub.kicad_sch (KiCad schematic)
At the start: 73 parts, among them IC19 USB5807C/KD, IC20 TPS62933ODRLR, Y2 VXM7-9032-25M0000000

Commit message: CM5_BOOT0 control modified
Parts:
- renumbered R61 to R62, R62 to R63, R63 to R64, R64 to R65, R65 to R66, R66 to R67, R67 to R68, R68 to R69, R69 to R70, R70 to R71, R71 to R72, R72 to R73, R73 to R74, R74 to R75, R75 to R76, R76 to R77, R77 to R78, R78 to R79
Changed lines of the file:
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@@
 		(in_pos_files yes)
 		(dnp no)
-		(property "Reference" "R78"
+		(property "Reference" "R79"
 			(at 246.38 156.21 90)
 			(show_name no)
@@
 			(project "BB3plus mainboard"
 				(path "/1df84e4f-233a-4f72-9418-c0020706bb76/99b67fa5-56ce-4798-a21a-d86c3d347c55"
-					(reference "R78")
+					(reference "R79")
 					(unit 1)
 				)
@@
 		(in_pos_files yes)
 		(dnp no)
-		(property "Reference" "R61"
+		(property "Reference" "R62"
 			(at 34.925 114.3 90)
 			(show_name no)
@@
 			(project "BB3plus mainboard"
 				(path "/1df84e4f-233a-4f72-9418-c0020706bb76/99b67fa5-56ce-4798-a21a-d86c3d347c55"
-					(reference "R61")
+					(reference "R62")
 					(unit 1)
 				)
@@
 		(in_pos_files yes)
 		(dnp no)
-		(property "Reference" "R70"
+		(property "Reference" "R71"
 			(at 46.355 71.12 90)
 			(show_name no)
@@
 			(project "BB3plus mainboard"
 				(path "/1df84e4f-233a-4f72-9418-c0020706bb76/99b67fa5-56ce-4798-a21a-d86c3d347c55"
-					(reference "R70")
+					(reference "R71")
 					(unit 1)
 				)
@@
 		(in_pos_files yes)
 		(dnp yes)
-		(property "Reference" "R62"
+		(property "Reference" "R63"
 			(at 40.64 95.25 90)
 			(show_name no)
@@
 			(project "BB3plus mainboard"
 				(path "/1df84e4f-233a-4f72-9418-c0020706bb76/99b67fa5-56ce-4798-a21a-d86c3d347c55"
-					(reference "R62")
+					(reference "R63")
 					(unit 1)
 				)
@@
 		(in_pos_files yes)
 		(dnp no)
-		(property "Reference" "R74"
+		(property "Reference" "R75"
 			(at 47.625 132.08 90)
 			(show_name no)
@@
 			(project "BB3plus mainboard"
 				(path "/1df84e4f-233a-4f72-9418-c0020706bb76/99b67fa5-56ce-4798-a21a-d86c3d347c55"
-					(reference "R74")
+					(reference "R75")
 					(unit 1)
 				)
@@
 		(in_pos_files yes)
 		(dnp no)
-		(property "Reference" "R75"
+		(property "Reference" "R76"
 			(at 168.91 156.21 90)
 			(show_name no)
@@
 			(project "BB3plus mainboard"
 				(path "/1df84e4f-233a-4f72-9418-c0020706bb76/99b67fa5-56ce-4798-a21a-d86c3d347c55"
-					(reference "R75")
+					(reference "R76")
 					(unit 1)
 				)
@@
 		(in_pos_files yes)
 		(dnp yes)
-		(property "Reference" "R63"
+		(property "Reference" "R64"
 			(at 50.8 21.59 90)
 			(show_name no)
@@
 			(project "BB3plus mainboard"
 				(path "/1df84e4f-233a-4f72-9418-c0020706bb76/99b67fa5-56ce-4798-a21a-d86c3d347c55"
-					(reference "R63")
+					(reference "R64")
 					(unit 1)
 				)
@@
 		(in_pos_files yes)
 		(dnp no)
-		(property "Reference" "R77"
+		(property "Reference" "R78"
 			(at 240.03 151.765 0)
 			(show_name no)
@@
 			(project "BB3plus mainboard"
 				(path "/1df84e4f-233a-4f72-9418-c0020706bb76/99b67fa5-56ce-4798-a21a-d86c3d347c55"
-					(reference "R77")
+					(reference "R78")
 					(unit 1)
 				)
@@
 		(in_pos_files yes)
 		(dnp no)
-		(property "Reference" "R69"
+		(property "Reference" "R70"
 			(at 46.355 68.58 90)
 			(show_name no)
@@
 			(project "BB3plus mainboard"
 				(path "/1df84e4f-233a-4f72-9418-c0020706bb76/99b67fa5-56ce-4798-a21a-d86c3d347c55"
-					(reference "R69")
+					(reference "R70")
 					(unit 1)
 				)
@@
 		(in_pos_files yes)
 		(dnp yes)
-		(property "Reference" "R64"
+		(property "Reference" "R65"
 			(at 50.8 29.21 90)
 			(show_name no)
@@
 			(project "BB3plus mainboard"
 				(path "/1df84e4f-233a-4f72-9418-c0020706bb76/99b67fa5-56ce-4798-a21a-d86c3d347c55"
-					(reference "R64")
+					(reference "R65")
 					(unit 1)
 				)
@@
 		(in_pos_files yes)
 		(dnp no)
-		(property "Reference" "R65"
+		(property "Reference" "R66"
 			(at 46.355 55.88 90)
 			(show_name no)
@@
 			(project "BB3plus mainboard"
 				(path "/1df84e4f-233a-4f72-9418-c0020706bb76/99b67fa5-56ce-4798-a21a-d86c3d347c55"
-					(reference "R65")
+					(reference "R66")
 					(unit 1)
 				)
@@
 		(in_pos_files yes)
 		(dnp no)
-		(property "Reference" "R68"
+		(property "Reference" "R69"
 			(at 46.355 63.5 90)
 			(show_name no)
@@
 			(project "BB3plus mainboard"
 				(path "/1df84e4f-233a-4f72-9418-c0020706bb76/99b67fa5-56ce-4798-a21a-d86c3d347c55"
-					(reference "R68")
+					(reference "R69")
 					(unit 1)
 				)
@@
 		(in_pos_files yes)
 		(dnp no)
-		(property "Reference" "R67"
+		(property "Reference" "R68"
 			(at 46.355 60.96 90)
 			(show_name no)
@@
 			(project "BB3plus mainboard"
 				(path "/1df84e4f-233a-4f72-9418-c0020706bb76/99b67fa5-56ce-4798-a21a-d86c3d347c55"
-					(reference "R67")
+					(reference "R68")
 					(unit 1)
 				)
@@
 		(in_pos_files yes)
 		(dnp no)
-		(property "Reference" "R66"
+		(property "Reference" "R67"
 			(at 46.355 58.42 90)
 			(show_name no)
@@
 			(project "BB3plus mainboard"
 				(path "/1df84e4f-233a-4f72-9418-c0020706bb76/99b67fa5-56ce-4798-a21a-d86c3d347c55"
-					(reference "R66")
+					(reference "R67")
 					(unit 1)
 				)
@@
 		(in_pos_files yes)
 		(dnp no)
-		(property "Reference" "R71"
+		(property "Reference" "R72"
 			(at 48.26 78.74 90)
 			(show_name no)
@@
 			(project "BB3plus mainboard"
 				(path "/1df84e4f-233a-4f72-9418-c0020706bb76/99b67fa5-56ce-4798-a21a-d86c3d347c55"
-					(reference "R71")
+					(reference "R72")
 					(unit 1)
 				)
@@
 		(in_pos_files yes)
 		(dnp no)
-		(property "Reference" "R73"
+		(property "Reference" "R74"
 			(at 47.625 127 90)
 			(show_name no)
@@
 			(project "BB3plus mainboard"
 				(path "/1df84e4f-233a-4f72-9418-c0020706bb76/99b67fa5-56ce-4798-a21a-d86c3d347c55"
-					(reference "R73")
+					(reference "R74")
 					(unit 1)
 				)
@@
 		(in_pos_files yes)
 		(dnp yes)
-		(property "Reference" "R72"
+		(property "Reference" "R73"
 			(at 50.8 92.71 90)
 			(show_name no)
@@
 			(project "BB3plus mainboard"
 				(path "/1df84e4f-233a-4f72-9418-c0020706bb76/99b67fa5-56ce-4798-a21a-d86c3d347c55"
-					(reference "R72")
+					(reference "R73")
 					(unit 1)
 				)
@@
 		(in_pos_files yes)
 		(dnp no)
-		(property "Reference" "R76"
+		(property "Reference" "R77"
 			(at 177.8 151.13 90)
 			(show_name no)
@@
 			(project "BB3plus mainboard"
 				(path "/1df84e4f-233a-4f72-9418-c0020706bb76/99b67fa5-56ce-4798-a21a-d86c3d347c55"
-					(reference "R76")
+					(reference "R77")
 					(unit 1)
 				)

Commit message: #21
Parts:
- renumbered C103 to C100, C104 to C101, C105 to C102, C106 to C103, C107 to C104, C108 to C105, C109 to C106, C110 to C107, C111 to C108, C112 to C109, C113 to C110, C70 to C67, C71 to C68, C72 to C69, C73 to C70, C74 to C71, C75 to C72, C76 to C73, C77 to C74, C78 to C75, C79 to C76, C80 to C77, C81 to C78, C82 to C79, C83 to C80, C84 to C81, C85 to C82, C86 to C83, C87 to C84, C88 to C85, C89 to C86, C90 to C87, C91 to C88, C92 to C89, C93 to C90, C94 to C91, C95 to C92, C96 to C93, C97 to C94, C98 to C95, C99 to C96, C100 to C97, C101 to C98, C102 to C99, IC19 to IC16, IC20 to IC17, JP11 to JP10, JP12 to JP11, JP13 to JP12, JP10 to JP9, L7 to L8, R62 to R60, R63 to R61, R64 to R62, R65 to R63, R66 to R64, R67 to R65, R68 to R66, R69 to R67, R70 to R68, R71 to R69, R72 to R70, R73 to R71, R74 to R72, R75 to R73, R76 to R74, R77 to R75, R78 to R76, R79 to R77, TP14 to TP12

Commit message: #22
Parts:
- renumbered JP9 to JP10, JP10 to JP11, JP11 to JP12, JP12 to JP13
Changed lines of the file:
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@@
 	(title_block
 		(title "${project_name}")
-		(date "2026-10-06")
+		(date "2026-10-08")
 		(rev "${project_version}")
 		(company "${project_creator}")
@@
 		(in_pos_files yes)
 		(dnp no)
-		(property "Reference" "#SUPPLY062"
+		(property "Reference" "#SUPPLY061"
 			(at 246.38 68.58 0)
 			(hide yes)
@@
 			(project "BB3plus mainboard"
 				(path "/1df84e4f-233a-4f72-9418-c0020706bb76/99b67fa5-56ce-4798-a21a-d86c3d347c55"
-					(reference "#SUPPLY062")
+					(reference "#SUPPLY061")
 					(unit 1)
 				)
@@
 		(in_pos_files yes)
 		(dnp no)
-		(property "Reference" "JP9"
+		(property "Reference" "JP10"
 			(at 22.86 144.78 90)
 			(show_name no)
@@
 			(project "BB3plus mainboard"
 				(path "/1df84e4f-233a-4f72-9418-c0020706bb76/99b67fa5-56ce-4798-a21a-d86c3d347c55"
-					(reference "JP9")
+					(reference "JP10")
 					(unit 1)
 				)
@@
 		(in_pos_files yes)
 		(dnp no)
-		(property "Reference" "#SUPPLY061"
+		(property "Reference" "#SUPPLY060"
 			(at 246.38 45.72 0)
 			(hide yes)
@@
 			(project "BB3plus mainboard"
 				(path "/1df84e4f-233a-4f72-9418-c0020706bb76/99b67fa5-56ce-4798-a21a-d86c3d347c55"
-					(reference "#SUPPLY061")
+					(reference "#SUPPLY060")
 					(unit 1)
 				)
@@
 		(in_pos_files yes)
 		(dnp no)
-		(property "Reference" "#SUPPLY060"
+		(property "Reference" "#SUPPLY059"
 			(at 226.06 88.9 0)
 			(hide yes)
@@
 			(project "BB3plus mainboard"
 				(path "/1df84e4f-233a-4f72-9418-c0020706bb76/99b67fa5-56ce-4798-a21a-d86c3d347c55"
-					(reference "#SUPPLY060")
+					(reference "#SUPPLY059")
 					(unit 1)
 				)
@@
 		(in_pos_files yes)
 		(dnp no)
-		(property "Reference" "#SUPPLY063"
+		(property "Reference" "#SUPPLY062"
 			(at 254 160.02 0)
 			(hide yes)
@@
 			(project "BB3plus mainboard"
 				(path "/1df84e4f-233a-4f72-9418-c0020706bb76/99b67fa5-56ce-4798-a21a-d86c3d347c55"
-					(reference "#SUPPLY063")
+					(reference "#SUPPLY062")
 					(unit 1)
 				)
@@
 		(in_pos_files yes)
 		(dnp no)
-		(property "Reference" "JP11"
+		(property "Reference" "JP12"
 			(at 40.64 102.87 0)
 			(show_name no)
@@
 			(project "BB3plus mainboard"
 				(path "/1df84e4f-233a-4f72-9418-c0020706bb76/99b67fa5-56ce-4798-a21a-d86c3d347c55"
-					(reference "JP11")
+					(reference "JP12")
 					(unit 1)
 				)
@@
 		(in_pos_files yes)
 		(dnp no)
-		(property "Reference" "#SUPPLY064"
+		(property "Reference" "#SUPPLY063"
 			(at 271.78 157.48 0)
 			(hide yes)
@@
 			(project "BB3plus mainboard"
 				(path "/1df84e4f-233a-4f72-9418-c0020706bb76/99b67fa5-56ce-4798-a21a-d86c3d347c55"
-					(reference "#SUPPLY064")
+					(reference "#SUPPLY063")
 					(unit 1)
 				)
@@
 		(in_pos_files yes)
 		(dnp no)
-		(property "Reference" "#SUPPLY059"
+		(property "Reference" "#SUPPLY058"
 			(at 213.36 157.48 0)
 			(hide yes)
@@
 			(project "BB3plus mainboard"
 				(path "/1df84e4f-233a-4f72-9418-c0020706bb76/99b67fa5-56ce-4798-a21a-d86c3d347c55"
-					(reference "#SUPPLY059")
+					(reference "#SUPPLY058")
 					(unit 1)
 				)
@@
 		(in_pos_files yes)
 		(dnp no)
-		(property "Reference" "#SUPPLY058"
+		(property "Reference" "#SUPPLY057"
 			(at 157.48 160.02 0)
 			(hide yes)
@@
 			(project "BB3plus mainboard"
 				(path "/1df84e4f-233a-4f72-9418-c0020706bb76/99b67fa5-56ce-4798-a21a-d86c3d347c55"
-					(reference "#SUPPLY058")
+					(reference "#SUPPLY057")
 					(unit 1)
 				)
@@
 		(in_pos_files yes)
 		(dnp no)
-		(property "Reference" "JP12"
+		(property "Reference" "JP13"
 			(at 173.99 69.85 0)
 			(show_name no)
@@
 			(project "BB3plus mainboard"
 				(path "/1df84e4f-233a-4f72-9418-c0020706bb76/99b67fa5-56ce-4798-a21a-d86c3d347c55"
-					(reference "JP12")
+					(reference "JP13")
 					(unit 1)
 				)
@@
 		(in_pos_files yes)
 		(dnp no)
-		(property "Reference" "JP10"
+		(property "Reference" "JP11"
 			(at 40.64 100.33 0)
 			(show_name no)
@@
 			(project "BB3plus mainboard"
 				(path "/1df84e4f-233a-4f72-9418-c0020706bb76/99b67fa5-56ce-4798-a21a-d86c3d347c55"
-					(reference "JP10")
+					(reference "JP11")
 					(unit 1)
 				)
