File: KiCad/BB3plus mainboard/usb_conn.kicad_sch (KiCad schematic)
At the start: 54 parts, among them IC21 MIC2026A-1YM-TR, IC22 PTN5150AHXMP, IC23 TPS2068E, IC24 TPD2E001DRLR, IC25 TPD2E001DRLR, IC26 FUSB340TMX, Q7 2N7002, Q8 2N7002, X14 USB4056-03-A, X15 MGB0A1-1CDDB005H

Commit message: CM5_BOOT0 control modified
Parts:
- added D16: BAS316, PCM_EEZ_SMD:SOD-323_1P8X1P35_ONS-M, symbol PCM_EEZ_discretes:DIODE
- renumbered R79 to R80, R80 to R81, R81 to R82, R82 to R83, R83 to R84, R84 to R85, R85 to R86, R86 to R87, R87 to R88, R88 to R89, R89 to R90, R90 to R91, R91 to R92
Connections:
- net at IC21.1 (ENA), R82.1: now also D16.A
- new net CM5_BOOT0: D16.C
Changed lines of the file:
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@@
 		(color 0 0 0 0)
 	)
+	(junction
+		(at 40.64 154.94)
+		(diameter 0)
+		(color 0 0 0 0)
+	)
 	(no_connect
 		(at 127 68.58)
@@
 	(wire
 		(pts
+			(xy 27.94 154.94) (xy 30.48 154.94)
+		)
+		(stroke
+			(width 0)
+			(type default)
+		)
+	)
+	(wire
+		(pts
 			(xy 203.2 60.96) (xy 208.28 60.96)
 		)
@@
 	(wire
 		(pts
+			(xy 35.56 154.94) (xy 40.64 154.94)
+		)
+		(stroke
+			(width 0)
+			(type default)
+		)
+	)
+	(wire
+		(pts
 			(xy 40.64 45.72) (xy 48.26 45.72)
 		)
@@
 		)
 	)
+	(global_label "CM5_BOOT0"
+		(shape input)
+		(at 27.94 154.94 180)
+		(fields_autoplaced yes)
+		(effects
+			(font
+				(size 0.889 0.889)
+			)
+			(justify right)
+		)
+		(property "Intersheetrefs" "${INTERSHEET_REFS}"
+			(at 18.6038 154.94 0)
+			(hide yes)
+			(show_name no)
+			(do_not_autoplace no)
+			(effects
+				(font
+					(size 1.27 1.27)
+				)
+				(justify right)
+			)
+		)
+	)
 	(global_label "REAR_USB_TOP_TX-"
 		(shape bidirectional)
@@
 		(in_pos_files yes)
 		(dnp no)
-		(property "Reference" "R84"
+		(property "Reference" "R85"
 			(at 60.96 125.73 90)
 			(show_name no)
@@
 			(project "BB3plus mainboard"
 				(path "/1df84e4f-233a-4f72-9418-c0020706bb76/c0a485a3-023d-4313-ae06-c16e1fdbf75a"
-					(reference "R84")
+					(reference "R85")
 					(unit 1)
 				)
@@
 		(in_pos_files yes)
 		(dnp no)
-		(property "Reference" "R89"
+		(property "Reference" "R90"
 			(at 224.79 75.565 0)
 			(show_name no)
@@
 			(project "BB3plus mainboard"
 				(path "/1df84e4f-233a-4f72-9418-c0020706bb76/c0a485a3-023d-4313-ae06-c16e1fdbf75a"
-					(reference "R89")
+					(reference "R90")
 					(unit 1)
 				)
@@
 		(in_pos_files yes)
 		(dnp no)
-		(property "Reference" "R85"
+		(property "Reference" "R86"
 			(at 60.96 138.43 90)
 			(show_name no)
@@
 			(project "BB3plus mainboard"
 				(path "/1df84e4f-233a-4f72-9418-c0020706bb76/c0a485a3-023d-4313-ae06-c16e1fdbf75a"
-					(reference "R85")
+					(reference "R86")
 					(unit 1)
 				)
@@
 		(in_pos_files yes)
 		(dnp no)
-		(property "Reference" "R81"
+		(property "Reference" "R82"
 			(at 41.91 147.32 0)
 			(show_name no)
@@
 			(project "BB3plus mainboard"
 				(path "/1df84e4f-233a-4f72-9418-c0020706bb76/c0a485a3-023d-4313-ae06-c16e1fdbf75a"
-					(reference "R81")
+					(reference "R82")
 					(unit 1)
 				)
@@
 	)
 	(symbol
+		(lib_id "PCM_EEZ_discretes:DIODE")
+		(at 33.02 154.94 180)
+		(unit 1)
+		(body_style 1)
+		(exclude_from_sim no)
+		(in_bom yes)
+		(on_board yes)
+		(in_pos_files yes)
+		(dnp no)
+		(property "Reference" "D16"
+			(at 33.02 153.035 0)
+			(show_name no)
+			(do_not_autoplace no)
+			(effects
+				(font
+					(size 1.27 1.27)
+				)
+				(justify top)
+			)
+		)
+		(property "Value" "BAS316"
+			(at 33.02 156.845 0)
+			(show_name no)
+			(do_not_autoplace no)
+			(effects
+				(font
+					(size 1.27 1.27)
+				)
+				(justify bottom)
+			)
+		)
+		(property "Footprint" "PCM_EEZ_SMD:SOD-323_1P8X1P35_ONS-M"
+			(at 33.02 151.765 0)
+			(hide yes)
+			(show_name no)
+			(do_not_autoplace no)
+			(effects
+				(font
+					(size 1.27 1.27)
+				)
+			)
+		)
+		(property "Datasheet" ""
+			(at 33.02 154.94 0)
+			(hide yes)
+			(show_name no)
+			(do_not_autoplace no)
+			(effects
+				(font
+					(size 1.27 1.27)
+				)
+			)
+		)
+		(property "Description" ""
+			(at 33.02 154.94 0)
+			(hide yes)
+			(show_name no)
+			(do_not_autoplace no)
+			(effects
+				(font
+					(size 1.27 1.27)
+				)
+			)
+		)
+		(property "DigiKey" "1727-7370-1-ND"
+			(at 33.02 154.94 0)
+			(hide yes)
+			(show_name no)
+			(do_not_autoplace no)
+			(effects
+				(font
+					(size 1.27 1.27)
+				)
+			)
+		)
+		(property "Mouser" "771-BAS316-T/R"
+			(at 33.02 154.94 0)
+			(hide yes)
+			(show_name no)
+			(do_not_autoplace no)
+			(effects
+				(font
+					(size 1.27 1.27)
+				)
+			)
+		)
+		(property "TME" "BAS316,115"
+			(at 33.02 154.94 0)
+			(hide yes)
+			(show_name no)
+			(do_not_autoplace no)
+			(effects
+				(font
+					(size 1.27 1.27)
+				)
+			)
+		)
+		(property "LCSC" "C2128"
+			(at 33.02 154.94 0)
+			(hide yes)
+			(show_name no)
+			(do_not_autoplace no)
+			(effects
+				(font
+					(size 1.27 1.27)
+				)
+			)
+		)
+		(pin "A"
+		)
+		(pin "C"
+		)
+		(instances
+			(project "BB3plus mainboard"
+				(path "/1df84e4f-233a-4f72-9418-c0020706bb76/c0a485a3-023d-4313-ae06-c16e1fdbf75a"
+					(reference "D16")
+					(unit 1)
+				)
+			)
+		)
+	)
+	(symbol
 		(lib_id "PCM_EEZ_symbols:GND")
 		(at 116.84 104.14 0)
@@
 		(in_pos_files yes)
 		(dnp no)
-		(property "Reference" "R80"
+		(property "Reference" "R81"
 			(at 36.83 147.32 0)
 			(show_name no)
@@
 			(project "BB3plus mainboard"
 				(path "/1df84e4f-233a-4f72-9418-c0020706bb76/c0a485a3-023d-4313-ae06-c16e1fdbf75a"
-					(reference "R80")
+					(reference "R81")
 					(unit 1)
 				)
@@
 		(in_pos_files yes)
 		(dnp no)
-		(property "Reference" "R83"
+		(property "Reference" "R84"
 			(at 59.69 30.48 0)
 			(show_name no)
@@
 			(project "BB3plus mainboard"
 				(path "/1df84e4f-233a-4f72-9418-c0020706bb76/c0a485a3-023d-4313-ae06-c16e1fdbf75a"
-					(reference "R83")
+					(reference "R84")
 					(unit 1)
 				)
@@
 		(in_pos_files yes)
 		(dnp no)
-		(property "Reference" "R82"
+		(property "Reference" "R83"
 			(at 49.53 30.48 0)
 			(show_name no)
@@
 			(project "BB3plus mainboard"
 				(path "/1df84e4f-233a-4f72-9418-c0020706bb76/c0a485a3-023d-4313-ae06-c16e1fdbf75a"
-					(reference "R82")
+					(reference "R83")
 					(unit 1)
 				)
@@
 		(in_pos_files yes)
 		(dnp no)
-		(property "Reference" "R87"
+		(property "Reference" "R88"
 			(at 132.08 100.33 90)
 			(show_name no)
@@
 			(project "BB3plus mainboard"
 				(path "/1df84e4f-233a-4f72-9418-c0020706bb76/c0a485a3-023d-4313-ae06-c16e1fdbf75a"
-					(reference "R87")
+					(reference "R88")
 					(unit 1)
 				)
@@
 		(in_pos_files yes)
 		(dnp no)
-		(property "Reference" "R91"
+		(property "Reference" "R92"
 			(at 273.05 137.16 0)
 			(show_name no)
@@
 			(project "BB3plus mainboard"
 				(path "/1df84e4f-233a-4f72-9418-c0020706bb76/c0a485a3-023d-4313-ae06-c16e1fdbf75a"
-					(reference "R91")
+					(reference "R92")
 					(unit 1)
 				)
@@
 		(in_pos_files yes)
 		(dnp no)
-		(property "Reference" "R90"
+		(property "Reference" "R91"
 			(at 255.27 137.16 0)
 			(show_name no)
@@
 			(project "BB3plus mainboard"
 				(path "/1df84e4f-233a-4f72-9418-c0020706bb76/c0a485a3-023d-4313-ae06-c16e1fdbf75a"
-					(reference "R90")
+					(reference "R91")
 					(unit 1)
 				)
@@
 		(in_pos_files no)
 		(dnp yes)
-		(property "Reference" "R79"
+		(property "Reference" "R80"
 			(at 35.56 74.93 90)
 			(show_name no)
@@
 			(project "BB3plus mainboard"
 				(path "/1df84e4f-233a-4f72-9418-c0020706bb76/c0a485a3-023d-4313-ae06-c16e1fdbf75a"
-					(reference "R79")
+					(reference "R80")
 					(unit 1)
 				)
@@
 		(in_pos_files yes)
 		(dnp no)
-		(property "Reference" "R86"
+		(property "Reference" "R87"
 			(at 121.92 100.33 90)
 			(show_name no)
@@
 			(project "BB3plus mainboard"
 				(path "/1df84e4f-233a-4f72-9418-c0020706bb76/c0a485a3-023d-4313-ae06-c16e1fdbf75a"
-					(reference "R86")
+					(reference "R87")
 					(unit 1)
 				)
@@
 		(in_pos_files no)
 		(dnp yes)
-		(property "Reference" "R88"
+		(property "Reference" "R89"
 			(at 147.32 34.29 90)
 			(show_name no)
@@
 			(project "BB3plus mainboard"
 				(path "/1df84e4f-233a-4f72-9418-c0020706bb76/c0a485a3-023d-4313-ae06-c16e1fdbf75a"
-					(reference "R88")
+					(reference "R89")
 					(unit 1)
 				)

Commit message: Mainboard 5V buck section modified
Parts:
- LED7: now in the parts list
Changed lines of the file:
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@@
 	(title_block
 		(title "${project_name}")
-		(date "2026-09-19")
+		(date "2026-10-04")
 		(rev "${project_version}")
 		(company "${project_creator}")
@@
 	(wire
 		(pts
-			(xy 93.98 157.48) (xy 93.98 162.56)
+			(xy 88.9 157.48) (xy 88.9 162.56)
 		)
 		(stroke
@@
 	(wire
 		(pts
-			(xy 93.98 162.56) (xy 149.86 162.56)
+			(xy 88.9 162.56) (xy 149.86 162.56)
 		)
 		(stroke
@@
 	(wire
 		(pts
-			(xy 78.74 157.48) (xy 93.98 157.48)
+			(xy 78.74 157.48) (xy 88.9 157.48)
 		)
 		(stroke
@@
 		(body_style 1)
 		(exclude_from_sim no)
-		(in_bom no)
+		(in_bom yes)
 		(on_board yes)
-		(in_pos_files no)
+		(in_pos_files yes)
 		(dnp yes)
 		(property "Reference" "LED7"

Commit message: #21
Parts:
- renumbered C114 to C111, C115 to C112, C116 to C113, C117 to C114, C118 to C115, C119 to C116, C120 to C117, C121 to C118, C122 to C119, C123 to C120, C124 to C121, C125 to C122, C126 to C123, C127 to C124, C128 to C125, C129 to C126, D16 to D14, IC21 to IC18, IC22 to IC19, IC23 to IC20, IC24 to IC21, IC25 to IC22, IC26 to IC23, JP14 to JP13, JP15 to JP14, JP16 to JP15, JP17 to JP16, L9 to L10, L10 to L11, L11 to L12, L8 to L9, R80 to R78, R81 to R79, R82 to R80, R83 to R81, R84 to R82, R85 to R83, R86 to R84, R87 to R85, R88 to R86, R89 to R87, R90 to R88, R91 to R89, R92 to R90, TP15 to TP13, TP16 to TP14, TP17 to TP15, TP18 to TP16

Commit message: #22
Parts:
- renumbered JP13 to JP14, JP14 to JP15, JP15 to JP16, JP16 to JP17
Changed lines of the file:
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@@
 	(title_block
 		(title "${project_name}")
-		(date "2026-10-06")
+		(date "2026-10-08")
 		(rev "${project_version}")
 		(company "${project_creator}")
@@
 		(in_pos_files yes)
 		(dnp no)
-		(property "Reference" "JP13"
+		(property "Reference" "JP14"
 			(at 59.69 67.31 0)
 			(show_name no)
@@
 			(project "BB3plus mainboard"
 				(path "/1df84e4f-233a-4f72-9418-c0020706bb76/c0a485a3-023d-4313-ae06-c16e1fdbf75a"
-					(reference "JP13")
+					(reference "JP14")
 					(unit 1)
 				)
@@
 		(in_pos_files yes)
 		(dnp no)
-		(property "Reference" "#SUPPLY066"
+		(property "Reference" "#SUPPLY065"
 			(at 177.8 73.66 0)
 			(hide yes)
@@
 			(project "BB3plus mainboard"
 				(path "/1df84e4f-233a-4f72-9418-c0020706bb76/c0a485a3-023d-4313-ae06-c16e1fdbf75a"
-					(reference "#SUPPLY066")
+					(reference "#SUPPLY065")
 					(unit 1)
 				)
@@
 		(in_pos_files yes)
 		(dnp no)
-		(property "Reference" "#SUPPLY068"
+		(property "Reference" "#SUPPLY067"
 			(at 205.74 73.66 0)
 			(hide yes)
@@
 			(project "BB3plus mainboard"
 				(path "/1df84e4f-233a-4f72-9418-c0020706bb76/c0a485a3-023d-4313-ae06-c16e1fdbf75a"
-					(reference "#SUPPLY068")
+					(reference "#SUPPLY067")
 					(unit 1)
 				)
@@
 		(in_pos_files yes)
 		(dnp no)
-		(property "Reference" "JP16"
+		(property "Reference" "JP17"
 			(at 59.69 90.17 0)
 			(show_name no)
@@
 			(project "BB3plus mainboard"
 				(path "/1df84e4f-233a-4f72-9418-c0020706bb76/c0a485a3-023d-4313-ae06-c16e1fdbf75a"
-					(reference "JP16")
+					(reference "JP17")
 					(unit 1)
 				)
@@
 		(in_pos_files yes)
 		(dnp no)
-		(property "Reference" "JP14"
+		(property "Reference" "JP15"
 			(at 59.69 72.39 0)
 			(show_name no)
@@
 			(project "BB3plus mainboard"
 				(path "/1df84e4f-233a-4f72-9418-c0020706bb76/c0a485a3-023d-4313-ae06-c16e1fdbf75a"
-					(reference "JP14")
+					(reference "JP15")
 					(unit 1)
 				)
@@
 		(in_pos_files yes)
 		(dnp no)
-		(property "Reference" "#SUPPLY065"
+		(property "Reference" "#SUPPLY064"
 			(at 177.8 43.18 0)
 			(hide yes)
@@
 			(project "BB3plus mainboard"
 				(path "/1df84e4f-233a-4f72-9418-c0020706bb76/c0a485a3-023d-4313-ae06-c16e1fdbf75a"
-					(reference "#SUPPLY065")
+					(reference "#SUPPLY064")
 					(unit 1)
 				)
@@
 		(in_pos_files yes)
 		(dnp no)
-		(property "Reference" "JP15"
+		(property "Reference" "JP16"
 			(at 59.69 77.47 0)
 			(show_name no)
@@
 			(project "BB3plus mainboard"
 				(path "/1df84e4f-233a-4f72-9418-c0020706bb76/c0a485a3-023d-4313-ae06-c16e1fdbf75a"
-					(reference "JP15")
+					(reference "JP16")
 					(unit 1)
 				)
@@
 		(in_pos_files yes)
 		(dnp no)
-		(property "Reference" "#SUPPLY067"
+		(property "Reference" "#SUPPLY066"
 			(at 205.74 43.18 0)
 			(hide yes)
@@
 			(project "BB3plus mainboard"
 				(path "/1df84e4f-233a-4f72-9418-c0020706bb76/c0a485a3-023d-4313-ae06-c16e1fdbf75a"
-					(reference "#SUPPLY067")
+					(reference "#SUPPLY066")
 					(unit 1)
 				)
