File: KiCad/BB3plus mainboard/dib.kicad_sch (KiCad schematic)
At the start: 5 parts, among them X19 1001878410201TLF, X20 1001878410201TLF, X21 1001878410201TLF, X22 1001878410201TLF, X23 1001878410201TLF

Commit message: #22
Connections:
- net +3V3: no longer X19.B15 (A0), X20.B16 (A1), X21.B15 (A0), X21.B16 (A1), X22.B17 (A2), X23.B15 (A0), X23.B17 (A2)
- net GND: now also X19.B15 (GND), X21.B15 (GND), X23.B15 (GND); no longer X19.B16 (A1), X19.B17 (A2), X20.B17 (A2), X21.B17 (A2), X22.B16 (A1), X23.B16 (A1)
- new net DIB1_REFCLK: X19.B17 (REFCLK+)
- new net DIB2_REFCLK: X20.B17 (REFCLK+)
- new net DIB3_REFCLK: X21.B17 (REFCLK+)
- new net DIB4_REFCLK: X22.B17 (REFCLK+)
- new net DIB5_REFCLK: X23.B17 (REFCLK+)
- no-connect marks 80 -> 85

Commit message: TOUT connected
Connections:
- net GND: no longer X19.B15 (GND), X20.B15 (GND), X21.B15 (GND), X22.B15 (GND), X23.B15 (GND)
- new net TOUT: X19.B15 (TOUT), X20.B15 (TOUT), X21.B15 (TOUT), X22.B15 (TOUT), X23.B15 (TOUT)
Changed lines of the file:
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@@
 	)
 	(junction
-		(at 106.68 137.16)
-		(diameter 0)
-		(color 0 0 0 0)
-	)
-	(junction
 		(at 58.42 99.06)
 		(diameter 0)
@@
 	)
 	(junction
-		(at 157.48 50.8)
-		(diameter 0)
-		(color 0 0 0 0)
-	)
-	(junction
 		(at 269.24 45.72)
 		(diameter 0)
@@
 	)
 	(junction
-		(at 210.82 106.68)
-		(diameter 0)
-		(color 0 0 0 0)
-	)
-	(junction
 		(at 25.4 45.72)
 		(diameter 0)
@@
 	)
 	(junction
-		(at 269.24 50.8)
-		(diameter 0)
-		(color 0 0 0 0)
-	)
-	(junction
 		(at 160.02 27.94)
 		(diameter 0)
@@
 	)
 	(junction
-		(at 58.42 50.8)
-		(diameter 0)
-		(color 0 0 0 0)
-	)
-	(junction
 		(at 236.22 35.56)
 		(diameter 0)
@@
 	(wire
 		(pts
+			(xy 271.78 58.42) (xy 266.7 58.42)
+		)
+		(stroke
+			(width 0)
+			(type default)
+		)
+	)
+	(wire
+		(pts
 			(xy 71.12 127) (xy 76.2 127)
 		)
@@
 	(wire
 		(pts
+			(xy 60.96 58.42) (xy 55.88 58.42)
+		)
+		(stroke
+			(width 0)
+			(type default)
+		)
+	)
+	(wire
+		(pts
 			(xy 271.78 53.34) (xy 266.7 53.34)
 		)
@@
 	(wire
 		(pts
-			(xy 106.68 137.16) (xy 106.68 144.78)
-		)
-		(stroke
-			(width 0)
-			(type default)
-		)
-	)
-	(wire
-		(pts
-			(xy 154.94 58.42) (xy 157.48 58.42)
-		)
-		(stroke
-			(width 0)
-			(type default)
-		)
-	)
-	(wire
-		(pts
 			(xy 175.26 96.52) (xy 180.34 96.52)
 		)
@@
 	(wire
 		(pts
+			(xy 213.36 114.3) (xy 208.28 114.3)
+		)
+		(stroke
+			(width 0)
+			(type default)
+		)
+	)
+	(wire
+		(pts
 			(xy 58.42 20.32) (xy 58.42 22.86)
 		)
@@
 	(wire
 		(pts
-			(xy 208.28 114.3) (xy 210.82 114.3)
-		)
-		(stroke
-			(width 0)
-			(type default)
-		)
-	)
-	(wire
-		(pts
 			(xy 25.4 76.2) (xy 27.94 76.2)
 		)
@@
 	(wire
 		(pts
-			(xy 55.88 58.42) (xy 58.42 58.42)
-		)
-		(stroke
-			(width 0)
-			(type default)
-		)
-	)
-	(wire
-		(pts
 			(xy 124.46 45.72) (xy 121.92 45.72)
 		)
@@
 	(wire
 		(pts
+			(xy 109.22 144.78) (xy 104.14 144.78)
+		)
+		(stroke
+			(width 0)
+			(type default)
+		)
+	)
+	(wire
+		(pts
 			(xy 213.36 93.98) (xy 208.28 93.98)
 		)
@@
 	(wire
 		(pts
-			(xy 210.82 106.68) (xy 210.82 114.3)
-		)
-		(stroke
-			(width 0)
-			(type default)
-		)
-	)
-	(wire
-		(pts
 			(xy 22.86 43.18) (xy 27.94 43.18)
 		)
@@
 	(wire
 		(pts
-			(xy 269.24 50.8) (xy 269.24 58.42)
-		)
-		(stroke
-			(width 0)
-			(type default)
-		)
-	)
-	(wire
-		(pts
 			(xy 177.8 83.82) (xy 180.34 83.82)
 		)
@@
 	(wire
 		(pts
-			(xy 104.14 144.78) (xy 106.68 144.78)
-		)
-		(stroke
-			(width 0)
-			(type default)
-		)
-	)
-	(wire
-		(pts
 			(xy 124.46 45.72) (xy 124.46 50.8)
 		)
@@
 	(wire
 		(pts
-			(xy 266.7 58.42) (xy 269.24 58.42)
-		)
-		(stroke
-			(width 0)
-			(type default)
-		)
-	)
-	(wire
-		(pts
 			(xy 60.96 38.1) (xy 55.88 38.1)
 		)
@@
 	(wire
 		(pts
-			(xy 58.42 50.8) (xy 58.42 58.42)
-		)
-		(stroke
-			(width 0)
-			(type default)
-		)
-	)
-	(wire
-		(pts
 			(xy 177.8 152.4) (xy 180.34 152.4)
 		)
@@
 	(wire
 		(pts
-			(xy 157.48 50.8) (xy 157.48 58.42)
-		)
-		(stroke
-			(width 0)
-			(type default)
-		)
-	)
-	(wire
-		(pts
 			(xy 236.22 78.74) (xy 238.76 78.74)
 		)
@@
 	(wire
 		(pts
+			(xy 160.02 58.42) (xy 154.94 58.42)
+		)
+		(stroke
+			(width 0)
+			(type default)
+		)
+	)
+	(wire
+		(pts
 			(xy 213.36 83.82) (xy 213.36 86.36)
 		)
@@
 		)
 	)
+	(global_label "TOUT"
+		(shape output)
+		(at 213.36 114.3 0)
+		(fields_autoplaced yes)
+		(effects
+			(font
+				(size 0.889 0.889)
+			)
+			(justify left)
+		)
+		(property "Intersheetrefs" "${INTERSHEET_REFS}"
+			(at 218.2088 114.3 0)
+			(hide yes)
+			(show_name no)
+			(do_not_autoplace no)
+			(effects
+				(font
+					(size 1.27 1.27)
+				)
+				(justify left)
+			)
+		)
+	)
 	(global_label "DIB1_USB_RX-"
 		(shape output)
@@
 		)
 	)
+	(global_label "TOUT"
+		(shape output)
+		(at 60.96 58.42 0)
+		(fields_autoplaced yes)
+		(effects
+			(font
+				(size 0.889 0.889)
+			)
+			(justify left)
+		)
+		(property "Intersheetrefs" "${INTERSHEET_REFS}"
+			(at 65.8088 58.42 0)
+			(hide yes)
+			(show_name no)
+			(do_not_autoplace no)
+			(effects
+				(font
+					(size 1.27 1.27)
+				)
+				(justify left)
+			)
+		)
+	)
 	(global_label "DIB_SCL"
 		(shape bidirectional)
@@
 		)
 	)
+	(global_label "TOUT"
+		(shape output)
+		(at 160.02 58.42 0)
+		(fields_autoplaced yes)
+		(effects
+			(font
+				(size 0.889 0.889)
+			)
+			(justify left)
+		)
+		(property "Intersheetrefs" "${INTERSHEET_REFS}"
+			(at 164.8688 58.42 0)
+			(hide yes)
+			(show_name no)
+			(do_not_autoplace no)
+			(effects
+				(font
+					(size 1.27 1.27)
+				)
+				(justify left)
+			)
+		)
+	)
 	(global_label "DIB1_USB_TX-"
 		(shape input)
@@
 		)
 	)
+	(global_label "TOUT"
+		(shape output)
+		(at 109.22 144.78 0)
+		(fields_autoplaced yes)
+		(effects
+			(font
+				(size 0.889 0.889)
+			)
+			(justify left)
+		)
+		(property "Intersheetrefs" "${INTERSHEET_REFS}"
+			(at 114.0688 144.78 0)
+			(hide yes)
+			(show_name no)
+			(do_not_autoplace no)
+			(effects
+				(font
+					(size 1.27 1.27)
+				)
+				(justify left)
+			)
+		)
+	)
 	(global_label "DIB1_USB_TX+"
 		(shape input)
@@
 			)
 		)
+	)
+	(global_label "TOUT"
+		(shape output)
+		(at 271.78 58.42 0)
+		(fields_autoplaced yes)
+		(effects
+			(font
+				(size 0.889 0.889)
+			)
+			(justify left)
+		)
+		(property "Intersheetrefs" "${INTERSHEET_REFS}"
+			(at 276.6288 58.42 0)
+			(hide yes)
+			(show_name no)
+			(do_not_autoplace no)
+			(effects
+				(font
+					(size 1.27 1.27)
+				)
+				(justify left)
+			)
+		)
