File: KiCad/BB3plus mainboard/dib.kicad_sch (KiCad schematic)
At the start: 5 parts, among them X19 1001878410201TLF, X20 1001878410201TLF, X21 1001878410201TLF, X22 1001878410201TLF, X23 1001878410201TLF

Commit message: Various small changes
Parts:
- X20: renamed from X19; value 1001878410201TLF -> 10018783-10101TLF
- X21: renamed from X20; value 1001878410201TLF -> 10018783-10101TLF
- X22: renamed from X21; value 1001878410201TLF -> 10018783-10101TLF
- X23: renamed from X22; value 1001878410201TLF -> 10018783-10101TLF
- X24: renamed from X23; value 1001878410201TLF -> 10018783-10101TLF
Changed lines of the file:
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@@
 	(title_block
 		(title "${project_name}")
-		(date "2026-10-09")
+		(date "2026-10-12")
 		(rev "${project_version}")
 		(company "${project_creator}")
@@
 		(in_pos_files yes)
 		(dnp no)
-		(property "Reference" "X19"
+		(property "Reference" "X20"
 			(at 34.925 16.51 0)
 			(show_name no)
@@
 			)
 		)
-		(property "Value" "1001878410201TLF"
+		(property "Value" "10018783-10101TLF"
 			(at 43.18 105.41 0)
 			(show_name no)
@@
 			(project "BB3plus mainboard"
 				(path "/1df84e4f-233a-4f72-9418-c0020706bb76/57aee854-8c94-4105-bcce-97e3d73b363b"
-					(reference "X19")
+					(reference "X20")
 					(unit 1)
 				)
@@
 		(in_pos_files yes)
 		(dnp no)
-		(property "Reference" "X23"
+		(property "Reference" "X24"
 			(at 245.745 16.51 0)
 			(show_name no)
@@
 			)
 		)
-		(property "Value" "1001878410201TLF"
+		(property "Value" "10018783-10101TLF"
 			(at 254 105.41 0)
 			(show_name no)
@@
 			(project "BB3plus mainboard"
 				(path "/1df84e4f-233a-4f72-9418-c0020706bb76/57aee854-8c94-4105-bcce-97e3d73b363b"
-					(reference "X23")
+					(reference "X24")
 					(unit 1)
 				)
@@
 		(in_pos_files yes)
 		(dnp no)
-		(property "Reference" "X21"
+		(property "Reference" "X22"
 			(at 133.985 16.51 0)
 			(show_name no)
@@
 			)
 		)
-		(property "Value" "1001878410201TLF"
+		(property "Value" "10018783-10101TLF"
 			(at 142.24 105.41 0)
 			(show_name no)
@@
 			(project "BB3plus mainboard"
 				(path "/1df84e4f-233a-4f72-9418-c0020706bb76/57aee854-8c94-4105-bcce-97e3d73b363b"
-					(reference "X21")
+					(reference "X22")
 					(unit 1)
 				)
@@
 		(in_pos_files yes)
 		(dnp no)
-		(property "Reference" "X22"
+		(property "Reference" "X23"
 			(at 187.325 72.39 0)
 			(show_name no)
@@
 			)
 		)
-		(property "Value" "1001878410201TLF"
+		(property "Value" "10018783-10101TLF"
 			(at 195.58 161.29 0)
 			(show_name no)
@@
 			(project "BB3plus mainboard"
 				(path "/1df84e4f-233a-4f72-9418-c0020706bb76/57aee854-8c94-4105-bcce-97e3d73b363b"
-					(reference "X22")
+					(reference "X23")
 					(unit 1)
 				)
@@
 		(in_pos_files yes)
 		(dnp no)
-		(property "Reference" "X20"
+		(property "Reference" "X21"
 			(at 83.185 102.87 0)
 			(show_name no)
@@
 			)
 		)
-		(property "Value" "1001878410201TLF"
+		(property "Value" "10018783-10101TLF"
 			(at 91.44 191.77 0)
 			(show_name no)
@@
 			(project "BB3plus mainboard"
 				(path "/1df84e4f-233a-4f72-9418-c0020706bb76/57aee854-8c94-4105-bcce-97e3d73b363b"
-					(reference "X20")
+					(reference "X21")
 					(unit 1)
 				)
