File: KiCad/BB3plus mainboard/dib.kicad_sch (KiCad schematic)
At the start: 5 parts, among them X20 10018783-10101TLF, X21 10018783-10101TLF, X22 10018783-10101TLF, X23 10018783-10101TLF, X24 10018783-10101TLF

Commit message: #28
Connections:
- removed net DIB_OE_SYNC: X20.B13 (OE_SNYC/TIN), X21.B13 (OE_SNYC/TIN), X22.B13 (OE_SNYC/TIN), X23.B13 (OE_SNYC/TIN), X24.B13 (OE_SNYC/TIN)
- removed net TOUT: X20.B15 (TOUT), X21.B15 (TOUT), X22.B15 (TOUT), X23.B15 (TOUT), X24.B15 (TOUT)
- new net DIB1_TIN: X20.B13 (OE_SNYC/TIN)
- new net DIB1_TOUT: X20.B15 (TOUT)
- new net DIB2_TIN: X21.B13 (OE_SNYC/TIN)
- new net DIB2_TOUT: X21.B15 (TOUT)
- new net DIB3_TIN: X22.B13 (OE_SNYC/TIN)
- new net DIB3_TOUT: X22.B15 (TOUT)
- new net DIB4_TIN: X23.B13 (OE_SNYC/TIN)
- new net DIB4_TOUT: X23.B15 (TOUT)
- new net DIB5_TIN: X24.B13 (OE_SNYC/TIN)
- new net DIB5_TOUT: X24.B15 (TOUT)
Changed lines of the file:
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@@
 	(title_block
 		(title "${project_name}")
-		(date "2026-10-18")
+		(date "2026-10-19")
 		(rev "${project_version}")
 		(company "${project_creator}")
@@
 		)
 	)
-	(global_label "~{DIB5_CSB}"
-		(shape input)
-		(at 236.22 86.36 180)
-		(fields_autoplaced yes)
-		(effects
-			(font
-				(size 0.889 0.889)
-			)
-			(justify right)
-		)
-		(property "Intersheetrefs" "${INTERSHEET_REFS}"
-			(at 228.2384 86.36 0)
-			(hide yes)
-			(show_name no)
-			(do_not_autoplace no)
-			(effects
-				(font
-					(size 1.27 1.27)
-				)
-				(justify right)
-			)
-		)
-	)
 	(global_label "~{DIB1_CSA}"
 		(shape input)
@@
 		)
 	)
-	(global_label "TOUT"
+	(global_label "DIB4_TOUT"
 		(shape output)
 		(at 213.36 114.3 0)
@@
 		)
 		(property "Intersheetrefs" "${INTERSHEET_REFS}"
-			(at 218.2088 114.3 0)
+			(at 221.9341 114.3 0)
 			(hide yes)
 			(show_name no)
@@
 		)
 	)
+	(global_label "~{DIB5_CSB}"
+		(shape input)
+		(at 236.22 86.36 180)
+		(fields_autoplaced yes)
+		(effects
+			(font
+				(size 0.889 0.889)
+			)
+			(justify right)
+		)
+		(property "Intersheetrefs" "${INTERSHEET_REFS}"
+			(at 228.2384 86.36 0)
+			(hide yes)
+			(show_name no)
+			(do_not_autoplace no)
+			(effects
+				(font
+					(size 1.27 1.27)
+				)
+				(justify right)
+			)
+		)
+	)
 	(global_label "DIB1_USB_RX-"
 		(shape output)
@@
 		)
 	)
-	(global_label "TOUT"
+	(global_label "DIB1_TOUT"
 		(shape output)
 		(at 60.96 58.42 0)
@@
 		)
 		(property "Intersheetrefs" "${INTERSHEET_REFS}"
-			(at 65.8088 58.42 0)
+			(at 69.5341 58.42 0)
 			(hide yes)
 			(show_name no)
@@
 		)
 	)
-	(global_label "DIB_OE_SYNC"
+	(global_label "DIB3_TIN"
 		(shape input)
 		(at 160.02 53.34 0)
@@
 		)
 		(property "Intersheetrefs" "${INTERSHEET_REFS}"
-			(at 170.3721 53.34 0)
+			(at 167.4088 53.34 0)
 			(hide yes)
 			(show_name no)
@@
 		)
 	)
-	(global_label "TOUT"
+	(global_label "DIB3_TOUT"
 		(shape output)
 		(at 160.02 58.42 0)
@@
 		)
 		(property "Intersheetrefs" "${INTERSHEET_REFS}"
-			(at 164.8688 58.42 0)
+			(at 168.5941 58.42 0)
 			(hide yes)
 			(show_name no)
@@
 		)
 	)
-	(global_label "DIB_OE_SYNC"
+	(global_label "DIB2_TIN"
 		(shape input)
 		(at 109.22 139.7 0)
@@
 		)
 		(property "Intersheetrefs" "${INTERSHEET_REFS}"
-			(at 119.5721 139.7 0)
+			(at 116.6088 139.7 0)
 			(hide yes)
 			(show_name no)
@@
 		)
 	)
-	(global_label "DIB_OE_SYNC"
+	(global_label "DIB5_TIN"
 		(shape input)
 		(at 271.78 53.34 0)
@@
 		)
 		(property "Intersheetrefs" "${INTERSHEET_REFS}"
-			(at 282.1321 53.34 0)
+			(at 279.1688 53.34 0)
 			(hide yes)
 			(show_name no)
@@
 		)
 	)
-	(global_label "TOUT"
+	(global_label "DIB2_TOUT"
 		(shape output)
 		(at 109.22 144.78 0)
@@
 		)
 		(property "Intersheetrefs" "${INTERSHEET_REFS}"
-			(at 114.0688 144.78 0)
+			(at 117.7941 144.78 0)
 			(hide yes)
 			(show_name no)
@@
 		)
 	)
-	(global_label "DIB_OE_SYNC"
+	(global_label "DIB1_TIN"
 		(shape input)
 		(at 60.96 53.34 0)
@@
 		)
 		(property "Intersheetrefs" "${INTERSHEET_REFS}"
-			(at 71.3121 53.34 0)
+			(at 68.3488 53.34 0)
 			(hide yes)
 			(show_name no)
@@
 		)
 	)
-	(global_label "DIB_OE_SYNC"
+	(global_label "DIB4_TIN"
 		(shape input)
 		(at 213.36 109.22 0)
@@
 		)
 		(property "Intersheetrefs" "${INTERSHEET_REFS}"
-			(at 223.7121 109.22 0)
+			(at 220.7488 109.22 0)
 			(hide yes)
 			(show_name no)
@@
 		)
 	)
-	(global_label "TOUT"
+	(global_label "DIB5_TOUT"
 		(shape output)
 		(at 271.78 58.42 0)
@@
 		)
 		(property "Intersheetrefs" "${INTERSHEET_REFS}"
-			(at 276.6288 58.42 0)
+			(at 280.3541 58.42 0)
 			(hide yes)
 			(show_name no)

Commit message: #29
Changed lines of the file:
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@@
 	(title_block
 		(title "${project_name}")
-		(date "2026-10-21")
+		(date "2026-10-22")
 		(rev "${project_version}")
 		(company "${project_creator}")
@@
 	)
 	(global_label "DIB5_REFCLK"
-		(shape bidirectional)
+		(shape input)
 		(at 271.78 63.5 0)
 		(fields_autoplaced yes)
@@
 		)
 		(property "Intersheetrefs" "${INTERSHEET_REFS}"
-			(at 282.7567 63.5 0)
+			(at 282.0899 63.5 0)
 			(hide yes)
 			(show_name no)
@@
 	)
 	(global_label "DIB4_REFCLK"
-		(shape input)
+		(shape bidirectional)
 		(at 213.36 119.38 0)
 		(fields_autoplaced yes)
@@
 		)
 		(property "Intersheetrefs" "${INTERSHEET_REFS}"
-			(at 223.6699 119.38 0)
+			(at 224.3367 119.38 0)
 			(hide yes)
 			(show_name no)
