File: KiCad/BB3plus mainboard/BB3plus mainboard.kicad_sch (KiCad schematic)
At the start: 19 parts

Commit message: #22
Other:
- sheet Ethernet, Video outputs renamed Ethernet, Video outputs, Ref clk
Changed lines of the file:
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@@
 	(title_block
 		(title "${project_name}")
-		(date "2026-10-06")
+		(date "2026-10-08")
 		(rev "${project_version}")
 		(company "${project_creator}")
@@
 			(color 0 0 0 0)
 		)
-		(property "Sheetname" "Ethernet, Video outputs"
+		(property "Sheetname" "Ethernet, Video outputs, Ref clk"
 			(at 60.96 42.4684 0)
 			(show_name no)
