File: KiCad/BB3plus mainboard/BB3plus mainboard.kicad_sch (KiCad schematic)
At the start: 19 parts

Commit message: #28
Other:
- sheet Power modules coupling renamed Trigger switch matrix, Power modules coupling
Changed lines of the file:
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@@
 	(title_block
 		(title "${project_name}")
-		(date "2026-10-18")
+		(date "2026-10-19")
 		(rev "${project_version}")
 		(company "${project_creator}")
@@
 		)
 		(column_widths 10.16 22.86)
-		(row_heights 2.54 2.54 2.54 2.54 2.54)
+		(row_heights 2.54 2.54 2.54 2.54 2.54 2.54)
 		(cells
 			(table_cell "I2C address"
@@
 				)
 			)
-			(table_cell "0x51"
+			(table_cell "0x53"
 				(exclude_from_sim no)
 				(at 25.4 96.52 0)
@@
 				)
 			)
+			(table_cell "0x70"
+				(exclude_from_sim no)
+				(at 25.4 106.68 0)
+				(size 10.16 2.54)
+				(margins 0.9525 0.9525 0.9525 0.9525)
+				(span 1 1)
+				(fill
+					(type none)
+				)
+				(effects
+					(font
+						(size 0.889 0.889)
+						(color 132 0 132 1)
+					)
+				)
+			)
+			(table_cell "ADG2188Y 8 x 8 switch array"
+				(exclude_from_sim no)
+				(at 35.56 106.68 0)
+				(size 22.86 2.54)
+				(margins 0.9525 0.9525 0.9525 0.9525)
+				(span 1 1)
+				(fill
+					(type none)
+				)
+				(effects
+					(font
+						(size 0.889 0.889)
+						(color 132 0 132 1)
+					)
+					(justify left)
+				)
+			)
 		)
 	)
@@
 			(color 0 0 0 0)
 		)
-		(property "Sheetname" "Power modules coupling"
+		(property "Sheetname" "Trigger switch matrix, Power modules coupling"
 			(at 137.16 42.4684 0)
 			(show_name no)
