File: KiCad/BB3plus mainboard/system_mcu.kicad_sch (KiCad schematic)
At the start: 61 parts, among them IC1 SN74HCS02PWR, IC2 M24C32-DFDW6TP, IC3 SN74LVC1G74DCUR, IC4 SN74LVC1G125DCKR, IC5 STM32G071R8T6, IC6 TPS3851H18EDRBR, IC7 SN74HCS02PWR, Q2 2N7002, Y1 FC-135 32.7680KA-K0

Commit message: #22
Parts:
- added JP8: (no value), PCM_EEZ_SMD:JP2 shorted (0603), symbol PCM_EEZ_unsorted:JP2 shorted
- renumbered C8 to C7, C7 to C8
Connections:
- net CM5_LED_PWR: now also IC5.11 (PF1-OSC_OUT); no longer IC5.10 (PF0-OSC_IN)
- new net: IC5.10 (PF0-OSC_IN), JP8.2
- new net SYSMCU_CLK: JP8.1
- no-connect marks 4 -> 3
Other:
- moved on the sheet: C7, D5, R12

Commit message: TOUT connected
Changed lines of the file:
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@@
 	(wire
 		(pts
-			(xy 35.56 137.16) (xy 35.56 147.32)
+			(xy 45.72 149.86) (xy 43.18 149.86)
 		)
 		(stroke
@@
 	(wire
 		(pts
-			(xy 45.72 149.86) (xy 43.18 149.86)
+			(xy 157.48 175.26) (xy 165.1 175.26)
 		)
 		(stroke
@@
 	(wire
 		(pts
-			(xy 157.48 175.26) (xy 165.1 175.26)
+			(xy 180.34 109.22) (xy 175.26 109.22)
 		)
 		(stroke
@@
 	(wire
 		(pts
-			(xy 180.34 109.22) (xy 175.26 109.22)
+			(xy 144.78 119.38) (xy 149.86 119.38)
 		)
 		(stroke
@@
 	(wire
 		(pts
-			(xy 144.78 119.38) (xy 149.86 119.38)
+			(xy 180.34 88.9) (xy 175.26 88.9)
 		)
 		(stroke
@@
 	(wire
 		(pts
-			(xy 180.34 88.9) (xy 175.26 88.9)
+			(xy 218.44 154.94) (xy 220.98 154.94)
 		)
 		(stroke
@@
 	(wire
 		(pts
-			(xy 218.44 154.94) (xy 220.98 154.94)
+			(xy 200.66 121.92) (xy 203.2 121.92)
 		)
 		(stroke
@@
 	(wire
 		(pts
-			(xy 200.66 121.92) (xy 203.2 121.92)
+			(xy 256.54 25.4) (xy 266.7 25.4)
+		)
+		(stroke
+			(width 0.1524)
+			(type solid)
+		)
+	)
+	(wire
+		(pts
+			(xy 124.46 165.1) (xy 124.46 170.18)
 		)
 		(stroke
@@
 	(wire
 		(pts
-			(xy 256.54 25.4) (xy 266.7 25.4)
+			(xy 144.78 116.84) (xy 149.86 116.84)
+		)
+		(stroke
+			(width 0)
+			(type default)
+		)
+	)
+	(wire
+		(pts
+			(xy 180.34 55.88) (xy 175.26 55.88)
+		)
+		(stroke
+			(width 0)
+			(type default)
+		)
+	)
+	(wire
+		(pts
+			(xy 200.66 121.92) (xy 200.66 111.76)
+		)
+		(stroke
+			(width 0)
+			(type default)
+		)
+	)
+	(wire
+		(pts
+			(xy 55.88 40.64) (xy 53.34 40.64)
+		)
+		(stroke
+			(width 0)
+			(type default)
+		)
+	)
+	(wire
+		(pts
+			(xy 276.86 71.12) (xy 269.24 71.12)
+		)
+		(stroke
+			(width 0)
+			(type default)
+		)
+	)
+	(wire
+		(pts
+			(xy 91.44 50.8) (xy 93.98 50.8)
+		)
+		(stroke
+			(width 0)
+			(type default)
+		)
+	)
+	(wire
+		(pts
+			(xy 220.98 35.56) (xy 220.98 40.64)
+		)
+		(stroke
+			(width 0)
+			(type default)
+		)
+	)
+	(wire
+		(pts
+			(xy 127 58.42) (xy 149.86 58.42)
+		)
+		(stroke
+			(width 0)
+			(type default)
+		)
+	)
+	(wire
+		(pts
+			(xy 50.8 48.26) (xy 53.34 48.26)
+		)
+		(stroke
+			(width 0)
+			(type default)
+		)
+	)
+	(wire
+		(pts
+			(xy 236.22 152.4) (xy 238.76 152.4)
+		)
+		(stroke
+			(width 0)
+			(type default)
+		)
+	)
+	(wire
+		(pts
+			(xy 269.24 86.36) (xy 269.24 83.82)
 		)
 		(stroke
@@
 	(wire
 		(pts
-			(xy 124.46 165.1) (xy 124.46 170.18)
+			(xy 175.26 50.8) (xy 187.96 50.8)
 		)
 		(stroke
@@
 	(wire
 		(pts
-			(xy 144.78 116.84) (xy 149.86 116.84)
+			(xy 111.76 99.06) (xy 111.76 109.22)
 		)
 		(stroke
@@
 	(wire
 		(pts
-			(xy 180.34 55.88) (xy 175.26 55.88)
+			(xy 144.78 167.64) (xy 142.24 167.64)
 		)
 		(stroke
@@
 	(wire
 		(pts
-			(xy 200.66 121.92) (xy 200.66 111.76)
+			(xy 124.46 109.22) (xy 127 109.22)
 		)
 		(stroke
@@
 	(wire
 		(pts
-			(xy 55.88 40.64) (xy 53.34 40.64)
+			(xy 116.84 58.42) (xy 119.38 58.42)
 		)
 		(stroke
@@
 	(wire
 		(pts
-			(xy 276.86 71.12) (xy 269.24 71.12)
+			(xy 254 93.98) (xy 251.46 93.98)
 		)
 		(stroke
@@
 	(wire
 		(pts
-			(xy 91.44 50.8) (xy 93.98 50.8)
+			(xy 25.4 147.32) (xy 45.72 147.32)
 		)
 		(stroke
@@
 	(wire
 		(pts
-			(xy 220.98 35.56) (xy 220.98 40.64)
+			(xy 162.56 160.02) (xy 162.56 165.1)
 		)
 		(stroke
@@
 	(wire
 		(pts
-			(xy 127 58.42) (xy 149.86 58.42)
-		)
-		(stroke
-			(width 0)
-			(type default)
-		)
-	)
-	(wire
-		(pts
-			(xy 50.8 48.26) (xy 53.34 48.26)
-		)
-		(stroke
-			(width 0)
-			(type default)
-		)
-	)
-	(wire
-		(pts
-			(xy 236.22 152.4) (xy 238.76 152.4)
-		)
-		(stroke
-			(width 0)
-			(type default)
-		)
-	)
-	(wire
-		(pts
-			(xy 269.24 86.36) (xy 269.24 83.82)
-		)
-		(stroke
-			(width 0.1524)
-			(type solid)
-		)
-	)
-	(wire
-		(pts
-			(xy 175.26 50.8) (xy 187.96 50.8)
-		)
-		(stroke
-			(width 0)
-			(type default)
-		)
-	)
-	(wire
-		(pts
-			(xy 111.76 99.06) (xy 111.76 109.22)
-		)
-		(stroke
-			(width 0)
-			(type default)
-		)
-	)
-	(wire
-		(pts
-			(xy 144.78 167.64) (xy 142.24 167.64)
-		)
-		(stroke
-			(width 0)
-			(type default)
-		)
-	)
-	(wire
-		(pts
-			(xy 124.46 109.22) (xy 127 109.22)
-		)
-		(stroke
-			(width 0)
-			(type default)
-		)
-	)
-	(wire
-		(pts
-			(xy 116.84 58.42) (xy 119.38 58.42)
-		)
-		(stroke
-			(width 0)
-			(type default)
-		)
-	)
-	(wire
-		(pts
-			(xy 254 93.98) (xy 251.46 93.98)
-		)
-		(stroke
-			(width 0)
-			(type default)
-		)
-	)
-	(wire
-		(pts
-			(xy 25.4 137.16) (xy 35.56 137.16)
-		)
-		(stroke
-			(width 0)
-			(type default)
-		)
-	)
-	(wire
-		(pts
-			(xy 162.56 160.02) (xy 162.56 165.1)
-		)
-		(stroke
-			(width 0)
-			(type default)
-		)
-	)
-	(wire
-		(pts
 			(xy 124.46 165.1) (xy 127 165.1)
-		)
-		(stroke
-			(width 0)
-			(type default)
-		)
-	)
-	(wire
-		(pts
-			(xy 35.56 147.32) (xy 45.72 147.32)
 		)
 		(stroke
@@
 		(row_heights 2.54 1.905 1.905 1.905 1.905)
 		(cells
-			(table_cell "~{BOOT_RST}"
+			(table_cell "DOUT1"
 				(exclude_from_sim no)
 				(at 181.61 149.86 0)
@@
 	(global_label "DIB_OE_SYNC"
 		(shape input)
-		(at 25.4 137.16 180)
-		(fields_autoplaced yes)
-		(effects
-			(font
-				(size 0.889 0.889)
-			)
-			(justify right)
-		)
-		(property "Intersheetrefs" "${INTERSHEET_REFS}"
-			(at 15.0479 137.16 0)
-			(hide yes)
-			(show_name no)
+		(at 25.4 147.32 180)
+		(fields_autoplaced yes)
+		(effects
+			(font
+				(size 0.889 0.889)
+			)
+			(justify right)
+		)
+		(property "Intersheetrefs" "${INTERSHEET_REFS}"
+			(at 15.0479 147.32 0)
+			(hide yes)
+			(show_name no)

Commit message: #23
Parts:
- IC5: value STM32G071R8T6 -> STM32G071RBT6; DigiKey 497-STM32G071R8T6-ND -> 497-18341-ND; LCSC C432214 -> C432213; Mouser 511-STM32G071R8T6 -> 511-STM32G071RBT6; TME STM32G071R8T6 -> STM32G071RBT6
Connections:
- net HUB_VBUS_EN: no longer names the net of IC5.40 (PD8)
- no-connect marks 3 -> 4
Changed lines of the file:
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@@
 	(title_block
 		(title "${project_name}")
-		(date "2026-10-08")
+		(date "2026-10-09")
 		(rev "${project_version}")
 		(company "${project_creator}")
@@
 	)
 	(no_connect
+		(at 149.86 124.46)
+	)
+	(no_connect
 		(at 218.44 68.58)
 	)
@@
 	(wire
 		(pts
-			(xy 144.78 124.46) (xy 149.86 124.46)
-		)
-		(stroke
-			(width 0)
-			(type default)
-		)
-	)
-	(wire
-		(pts
 			(xy 269.24 71.12) (xy 269.24 76.2)
 		)
@@
 		)
 	)
-	(global_label "HUB_VBUS_EN"
-		(shape output)
-		(at 144.78 124.46 180)
-		(fields_autoplaced yes)
-		(effects
-			(font
-				(size 0.889 0.889)
-				(color 204 102 0 1)
-			)
-			(justify right)
-		)
-		(property "Intersheetrefs" "${INTERSHEET_REFS}"
-			(at 133.8776 124.46 0)
-			(hide yes)
-			(show_name no)
-			(do_not_autoplace no)
-			(effects
-				(font
-					(size 1.27 1.27)
-				)
-				(justify right)
-			)
-		)
-	)
 	(global_label "FLEX_CMD"
 		(shape output)
@@
 			)
 		)
-		(property "Value" "STM32G071R8T6"
+		(property "Value" "STM32G071RBT6"
 			(at 152.4 130.175 0)
 			(show_name no)
@@
 			)
 		)
-		(property "DigiKey" "497-STM32G071R8T6-ND"
+		(property "DigiKey" "497-18341-ND"
 			(at 149.86 139.7 0)
 			(hide yes)
@@
 			)
 		)
-		(property "Mouser" "511-STM32G071R8T6"
+		(property "Mouser" "511-STM32G071RBT6"
 			(at 149.86 142.24 0)
 			(hide yes)
@@
 			)
 		)
-		(property "TME" "STM32G071R8T6"
+		(property "TME" "STM32G071RBT6"
 			(at 149.86 144.78 0)
 			(hide yes)
@@
 			)
 		)
-		(property "LCSC" "C432214"
+		(property "LCSC" "C432213"
 			(at 149.86 147.32 0)
 			(hide yes)

Commit message: #24
Parts:
- removed C12, C4: 100n, PCM_EEZ_passives:C_0603_1608Metric, symbol PCM_EEZ_passives:C-EU
- removed D1, D2, D3, D4, D6, D7: BAS316, PCM_EEZ_SMD:SOD-323_1P8X1P35_ONS-M, symbol PCM_EEZ_discretes:DIODE
- removed IC1: SN74HCS02PWR, PCM_EEZ_SMD:TSSOP-14, symbol PCM_EEZ_TI:SN74HCS02PWR
- removed IC3: SN74LVC1G74DCUR, PCM_EEZ_SMD:DCU8, symbol PCM_EEZ_TI:SN74LVC1G74DCUR
- removed IC4: SN74LVC1G125DCKR, PCM_EEZ_SMD:SOT65P210X110-5N, symbol PCM_EEZ_TI:SN74LVC1G125DCKR
- removed JP7: (no value), PCM_EEZ_SMD:JP3 shorted (0603), symbol PCM_EEZ_unsorted:JP3 shorted
- removed R14, R8, R9: 10K, PCM_EEZ_passives:R_0603_1608Metric, symbol PCM_EEZ_passives:R-EU
- renumbered C13 to C12, C14 to C13, C16 to C14, C3 to C2, C15 to C3, C2 to C4, D5 to D1, D8 to D2, D9 to D3, IC2 to IC1, IC6 to IC2, IC5 to IC3, IC7 to IC4, JP8 to JP7, R26 to R12, R12 to R13, R13 to R14, R23 to R21, R24 to R22, R25 to R23, R21 to R8, R22 to R9, TP3 to TP2, TP2 to TP3
Connections:
- net ~{DIB_SD_SYSMCU} is gone; now on net ~{DIB_SHUTDOWN}: IC3.59 (PB5)
- net ~{RPI_PWR_ON} is gone; now on net ~{CM5_PWR_BTN}: IC3.20 (PA3)
Other:
- note removed: "SYSMCU bootloader control"
- moved on the sheet: C10, C11, C12, C13, C14, C2, C3, C4, C5, C6, C7, C8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

Commit message: USB CC wiring updated
Parts:
- R14: value 750R -> 1K; DigiKey RC0603FR-07750RL -> 13-RC0603FR-131KLCT-ND; LCSC C23241 -> C21190; Mouser 603-RC0603FR-07750RL -> 603-RC0603FR-131KL; TME SMD0603-750R-1% -> CQ0603-1K-1%
Connections:
- net USBC_PORT_ROLE: no longer names the net of IC3.28 (PB1)
- no-connect marks 4 -> 5
Changed lines of the file:
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@@
 	(title_block
 		(title "${project_name}")
-		(date "2026-10-12")
+		(date "2026-10-14")
 		(rev "${project_version}")
 		(company "${project_creator}")
@@
 	)
 	(no_connect
+		(at 170.18 101.6)
+	)
+	(no_connect
 		(at 213.36 83.82)
 	)
@@
 	(wire
 		(pts
-			(xy 170.18 101.6) (xy 175.26 101.6)
-		)
-		(stroke
-			(width 0)
-			(type default)
-		)
-	)
-	(wire
-		(pts
 			(xy 30.48 40.64) (xy 33.02 40.64)
 		)
@@
 		)
 	)
-	(global_label "USBC_PORT_ROLE"
-		(shape output)
-		(at 175.26 101.6 0)
-		(fields_autoplaced yes)
-		(effects
-			(font
-				(size 0.889 0.889)
-				(color 204 102 0 1)
-			)
-			(justify left)
-		)
-		(property "Intersheetrefs" "${INTERSHEET_REFS}"
-			(at 188.5331 101.6 0)
-			(hide yes)
-			(show_name no)
-			(do_not_autoplace no)
-			(effects
-				(font
-					(size 1.27 1.27)
-				)
-				(justify left)
-			)
-		)
-	)
 	(global_label "SYS_SDA"
 		(shape bidirectional)
@@
 			)
 		)
-		(property "Value" "750R"
+		(property "Value" "1K"
 			(at 124.46 138.43 90)
 			(show_name no)
@@
 			)
 		)
-		(property "DigiKey" "RC0603FR-07750RL"
+		(property "DigiKey" "13-RC0603FR-131KLCT-ND"
 			(at 124.46 137.16 0)
 			(hide yes)
@@
 			)
 		)
-		(property "Mouser" "603-RC0603FR-07750RL"
+		(property "Mouser" "603-RC0603FR-131KL"
 			(at 124.46 137.16 0)
 			(hide yes)
@@
 			)
 		)
-		(property "TME" "SMD0603-750R-1%"
+		(property "TME" "CQ0603-1K-1%"
 			(at 124.46 137.16 0)
 			(hide yes)
@@
 			)
 		)
-		(property "LCSC" "C23241"
+		(property "LCSC" "C21190"
 			(at 124.46 137.16 0)
 			(hide yes)

Commit message: DVID_PWR_FAULT added
Connections:
- net ~{DVID_PWR_FAULT}: now reaches IC3.40 (PD8)
- no-connect marks 5 -> 4
Changed lines of the file:
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@@
 	)
 	(no_connect
-		(at 144.78 139.7)
-	)
-	(no_connect
 		(at 170.18 101.6)
 	)
@@
 	(wire
 		(pts
+			(xy 139.7 139.7) (xy 144.78 139.7)
+		)
+		(stroke
+			(width 0)
+			(type default)
+		)
+	)
+	(wire
+		(pts
 			(xy 170.18 132.08) (xy 175.26 132.08)
 		)
@@
 			)
 		)
+	)
+	(global_label "~{DVID_PWR_FAULT}"
+		(shape input)
+		(at 139.7 139.7 180)
+		(fields_autoplaced yes)
+		(effects
+			(font
+				(size 0.889 0.889)
+				(color 255 153 0 1)
+			)
+			(justify right)
+		)
+		(property "Intersheetrefs" "${INTERSHEET_REFS}"
+			(at 127.1042 139.7 0)
+			(hide yes)
+			(show_name no)
+			(do_not_autoplace no)
+			(effects
+				(font
+					(size 1.27 1.27)
+				)
+				(justify right)
+			)
+		)
