File: KiCad/BB3plus mainboard/system_mcu.kicad_sch (KiCad schematic)
At the start: 47 parts, among them IC1 M24C32-DFDW6TP, IC2 TPS3851H18EDRBR, IC3 STM32G071RBT6, IC4 SN74HCS02PWR, Q2 2N7002, Y1 FC-135 32.7680KA-K0

Commit message: DVID_PWR_ON added
Connections:
- net +3V3: now also IC1.2 (A1); no longer IC1.1 (A0)
- net ~{DIB_SHUTDOWN}: now also IC3.28 (PB1); no longer IC3.59 (PB5)
- net ~{USBC_IRQ}: now also IC3.59 (PB5); no longer IC3.53 (PD3)
- net at JP6.COM: now also IC1.1 (A0); no longer IC1.2 (A1)
- new net DVID_PWR_ON: IC3.53 (PD3)
- no-connect marks 4 -> 3
Other:
- moved on the sheet: C4, JP6

Commit message: SYSMCU pinout updated
Connections:
- net CM5_LED_PWR: now also IC3.3 (PC13); no longer IC3.11 (PF1-OSC_OUT)
- net SOFT_PWR: now also IC3.15 (PC2); no longer IC3.32 (PB12)
- net USBC_CONN_DET: now also IC3.32 (PB12); no longer IC3.15 (PC2)
- net ~{DIB1_CSB}: now also IC3.11 (PF1-OSC_OUT); no longer IC3.3 (PC13)
- net ~{DIB1_RESET}: now also IC3.55 (PD5); no longer IC3.54 (PD4)
- net ~{POWER_SW}: now also IC3.54 (PD4); no longer IC3.55 (PD5)
Other:
- note added: "RTC freq fanout"
- moved on the sheet: D2, IC4A, IC4B, IC4C, R21, R22, TP3

Commit message: Rear USB & Ethernet updated
Parts:
- added TP2, TP3: PCB_TEST_TABSHIELD, PCM_EEZ_THT:Testhole 12_25mils, symbol PCM_EEZ_unsorted:PCB test point
- renumbered C4 to C3, C3 to C4, TP2 to TP4, TP3 to TP5
Connections:
- net SYS_SCL: now also TP2.1 (P$1)
- net SYS_SDA: now also TP3.1 (P$1)
- net CM5_BOOT0 renamed CM5_BOOT

Commit message: #28
Connections:
- net +3V3: now also IC1.1 (A0)
- net GND: no longer IC1.3 (A2)
- net at JP6.COM: now also IC1.3 (A2); no longer IC1.1 (A0)
Other:
- moved on the sheet: JP6
Changed lines of the file:
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@@
 	(title_block
 		(title "${project_name}")
-		(date "2026-10-18")
+		(date "2026-10-19")
 		(rev "${project_version}")
 		(company "${project_creator}")
@@
 		)
 	)
-	(text_box "Mainboard ID: 002 (changeable to 011)"
+	(text_box "Mainboard ID: 003 (changeable to 100)"
 		(exclude_from_sim no)
-		(at 64.135 39.37 0)
+		(at 66.675 39.37 0)
 		(size 17.78 7.62)
 		(margins 0.9525 0.9525 0.9525 0.9525)
@@
 	)
 	(junction
-		(at 66.04 48.26)
-		(diameter 0)
-		(color 0 0 0 0)
-	)
-	(junction
 		(at 60.96 33.02)
 		(diameter 0)
@@
 	)
 	(junction
+		(at 60.96 43.18)
+		(diameter 0)
+		(color 0 0 0 0)
+	)
+	(junction
 		(at 132.08 30.48)
 		(diameter 0)
@@
 	(wire
 		(pts
+			(xy 58.42 48.26) (xy 63.5 48.26)
+		)
+		(stroke
+			(width 0)
+			(type default)
+		)
+	)
+	(wire
+		(pts
 			(xy 182.88 81.28) (xy 170.18 81.28)
 		)
@@
 	(wire
 		(pts
+			(xy 63.5 43.18) (xy 63.5 48.26)
+		)
+		(stroke
+			(width 0)
+			(type default)
+		)
+	)
+	(wire
+		(pts
 			(xy 139.7 106.68) (xy 144.78 106.68)
 		)
@@
 	(wire
 		(pts
-			(xy 60.96 38.1) (xy 60.96 45.72)
+			(xy 60.96 38.1) (xy 60.96 43.18)
 		)
 		(stroke
@@
 	(wire
 		(pts
-			(xy 66.04 38.1) (xy 66.04 40.64)
+			(xy 68.58 38.1) (xy 68.58 40.64)
 		)
 		(stroke
@@
 	(wire
 		(pts
+			(xy 58.42 43.18) (xy 60.96 43.18)
+		)
+		(stroke
+			(width 0)
+			(type default)
+		)
+	)
+	(wire
+		(pts
 			(xy 170.18 116.84) (xy 203.2 116.84)
 		)
@@
 	(wire
 		(pts
-			(xy 66.04 48.26) (xy 66.04 50.8)
-		)
-		(stroke
-			(width 0)
-			(type default)
-		)
-	)
-	(wire
-		(pts
 			(xy 233.68 106.68) (xy 236.22 106.68)
 		)
@@
 	(wire
 		(pts
-			(xy 66.04 45.72) (xy 66.04 48.26)
+			(xy 68.58 45.72) (xy 68.58 50.8)
 		)
 		(stroke
@@
 	(wire
 		(pts
-			(xy 60.96 38.1) (xy 66.04 38.1)
+			(xy 60.96 38.1) (xy 68.58 38.1)
 		)
 		(stroke
@@
 	(wire
 		(pts
-			(xy 58.42 48.26) (xy 66.04 48.26)
-		)
-		(stroke
-			(width 0)
-			(type default)
-		)
-	)
-	(wire
-		(pts
 			(xy 256.54 43.18) (xy 256.54 45.72)
 		)
@@
 	(wire
 		(pts
+			(xy 63.5 43.18) (xy 66.04 43.18)
+		)
+		(stroke
+			(width 0)
+			(type default)
+		)
+	)
+	(wire
+		(pts
 			(xy 124.46 38.1) (xy 132.08 38.1)
 		)
@@
 	(wire
 		(pts
+			(xy 60.96 43.18) (xy 60.96 45.72)
+		)
+		(stroke
+			(width 0)
+			(type default)
+		)
+	)
+	(wire
+		(pts
 			(xy 175.26 129.54) (xy 170.18 129.54)
 		)
@@
 	(wire
 		(pts
-			(xy 58.42 43.18) (xy 63.5 43.18)
-		)
-		(stroke
-			(width 0)
-			(type default)
-		)
-	)
-	(wire
-		(pts
 			(xy 223.52 43.18) (xy 223.52 45.72)
 		)
@@
 	(symbol
 		(lib_id "power:GND")
-		(at 66.04 50.8 0)
+		(at 68.58 50.8 0)
 		(mirror y)
 		(unit 1)
@@
 		(dnp no)
 		(property "Reference" "#GND02"
-			(at 66.04 50.8 0)
+			(at 68.58 50.8 0)
 			(hide yes)
 			(show_name no)
@@
 		)
 		(property "Value" "GND"
-			(at 69.85 51.435 0)
+			(at 72.39 51.435 0)
 			(show_name no)
 			(do_not_autoplace no)
@@
 		)
 		(property "Footprint" ""
-			(at 66.04 50.8 0)
+			(at 68.58 50.8 0)
 			(hide yes)
 			(show_name no)
@@
 		)
 		(property "Datasheet" ""
-			(at 66.04 50.8 0)
+			(at 68.58 50.8 0)
 			(hide yes)
 			(show_name no)
@@
 		)
 		(property "Description" "Power symbol creates a global label with name \"GND\" , ground"
-			(at 66.04 50.8 0)
+			(at 68.58 50.8 0)
 			(hide yes)
 			(show_name no)
@@
 	(symbol
 		(lib_id "PCM_EEZ_unsorted:JP3 shorted")
-		(at 66.04 43.18 0)
+		(at 68.58 43.18 0)
 		(mirror y)
 		(unit 1)
@@
 		(dnp no)
 		(property "Reference" "JP6"
-			(at 66.675 42.545 0)
+			(at 69.215 42.545 0)
 			(show_name no)
 			(do_not_autoplace no)
@@
 		)
 		(property "Value" ""
-			(at 66.04 43.18 0)
+			(at 68.58 43.18 0)
 			(hide yes)
 			(show_name no)
@@
 		)
 		(property "Footprint" "PCM_EEZ_SMD:JP3 shorted (0603)"
-			(at 66.04 48.26 0)
+			(at 68.58 48.26 0)
 			(hide yes)
 			(show_name no)
@@
 		)
 		(property "Datasheet" ""
-			(at 66.04 43.18 0)
+			(at 68.58 43.18 0)
 			(hide yes)
 			(show_name no)
@@
 		)
 		(property "Description" ""
-			(at 66.04 43.18 0)
+			(at 68.58 43.18 0)
 			(hide yes)
 			(show_name no)
@@
 		)
 		(property "DigiKey" ""
-			(at 66.04 43.18 0)
+			(at 68.58 43.18 0)
 			(hide yes)
 			(show_name no)
@@
 		)
 		(property "Mouser" ""
-			(at 66.04 43.18 0)
+			(at 68.58 43.18 0)
 			(hide yes)
 			(show_name no)
@@
 		)
 		(property "TME" ""
-			(at 66.04 43.18 0)
+			(at 68.58 43.18 0)
 			(hide yes)
 			(show_name no)
@@
 		)
 		(property "LCSC" ""
-			(at 66.04 43.18 0)
+			(at 68.58 43.18 0)
 			(hide yes)
 			(show_name no)
@@
 		)
 		(property "MF" ""
-			(at 66.04 43.18 0)
+			(at 68.58 43.18 0)
 			(hide yes)
 			(show_name no)
@@
 		)
 		(property "MP" ""
-			(at 66.04 43.18 0)
+			(at 68.58 43.18 0)
 			(hide yes)
 			(show_name no)
@@
 		)
 		(property "Name" ""
-			(at 66.04 43.18 0)
+			(at 68.58 43.18 0)
 			(hide yes)
 			(show_name no)
@@
 		)
 		(property "PN" ""
-			(at 66.04 43.18 0)
+			(at 68.58 43.18 0)
 			(hide yes)
 			(show_name no)

Commit message: #29
Parts:
- X4: footprint PCM_EEZ_connectors:WR-WST_490107670612_DEBUG -> PCM_EEZ_connectors:WR-WST_490107670612_DEBUG_pads
Changed lines of the file:
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@@
 	(title_block
 		(title "${project_name}")
-		(date "2026-10-21")
+		(date "2026-10-22")
 		(rev "${project_version}")
 		(company "${project_creator}")
@@
 			)
 		)
-		(property "Footprint" "PCM_EEZ_connectors:WR-WST_490107670612_DEBUG"
+		(property "Footprint" "PCM_EEZ_connectors:WR-WST_490107670612_DEBUG_pads"
 			(at 210.82 101.6 0)
 			(hide yes)
