File: KiCad/BB3plus mainboard/video_outputs.kicad_sch (KiCad schematic)
At the start: 22 parts, among them IC24 TPS22948DCKR, X15 MGB0A1-1CDDB005H, X16 SS-53000-002, X17 505110-2291, X18 505110-2291

Commit message: #22
Parts:
- added C133: 10u, PCM_EEZ_passives:C_0805_2012Metric, symbol PCM_EEZ_passives:C-EU
- added C134: 1u, PCM_EEZ_passives:C_0603_1608Metric, symbol PCM_EEZ_passives:C-EU
- added C135, C136, C137: 100n, PCM_EEZ_passives:C_0402_1005Metric, symbol PCM_EEZ_passives:C-EU
- added FB6: 60R@100MHz, PCM_EEZ_passives:BEAD0603, symbol PCM_EEZ_passives:L_Ferrite Bead
- added IC25, IC27: SN74LVC1G3157DCK, PCM_EEZ_SMD:SOT65P210X110-6N, symbol PCM_EEZ_TI:SN74LVC1G3157DCK
- added IC26: LMK1C1106APWR, PCM_EEZ_SMD:SOP65P640X120-14N, symbol PCM_EEZ_TI:LMK1C1106APWR
- added JP18: 10129378-902001BLF, PCM_EEZ_connectors:PinHeader_1x02_P2.54mm_Vertical, symbol PCM_EEZ_unsorted:JP2 open 2.54mm THT
- added R95: 47K, PCM_EEZ_passives:R_0603_1608Metric, symbol PCM_EEZ_passives:R-EU
- added Y3: ECS-TXO-32CSMV-100-AN-TR, PCM_EEZ_passives:XTAL_403C11A24M00000, symbol PCM_EEZ_passives:ECS-TXO-32CSMV-100-AN-TR
- renumbered JP17 to JP19
Connections:
- net +3V3: now also C133.1, FB6.1, IC25.5 (VDD), IC27.5 (VDD), JP18.2
- net GND: now also C133.2, C134.2, C135.2, C136.2, C137.2, IC25.2 (GND), IC26.10 (GND), IC26.4 (GND), IC26.7 (GND), IC27.2 (GND), R95.2, Y3.1 (GND), Y3.2 (GND)
- new net: IC25.1 (NO), IC27.1 (NO)
- new net: IC26.3 (Y0), IC27.3 (NC)
- new net: IC25.3 (NC), Y3.3 (Out)
- new net: IC25.4 (COM), IC26.1 (CLKIN)
- new net CLK_VDD: C134.1, C135.1, C136.1, C137.1, FB6.2, IC26.12 (VDD), IC26.2 (1G), IC26.5 (VDD), IC26.8 (VDD), Y3.4 (Vdd)
- new net DIB1_REFCLK: IC26.9 (Y5)
- new net DIB2_REFCLK: IC26.11 (Y2)
- new net DIB3_REFCLK: IC26.13 (Y3)
- new net DIB4_REFCLK: IC26.14 (Y1)
- new net DIB5_REFCLK: IC27.4 (COM)
- new net REFCLK #5: IC25.6 (CTRL), IC27.6 (CTRL), JP18.1, R95.1
- new net SYSMCU_CLK: IC26.6 (Y4)
Other:
- note added: "10MHz refclk & fanout"
- moved on the sheet: JP19, X17, X18

Commit message: PE fault detection section updated
Parts:
- renumbered C127 to C128, C128 to C129, C129 to C130, C130 to C131, C131 to C132, C132 to C133, C133 to C134, C134 to C135, C135 to C136, C136 to C137, C137 to C138, JP18 to JP20, JP19 to JP21

Commit message: Various small changes
Parts:
- renumbered X15 to X16, X16 to X17, X17 to X18, X18 to X19
Changed lines of the file:
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@@
 	(title_block
 		(title "${project_name}")
-		(date "2026-10-09")
+		(date "2026-10-12")
 		(rev "${project_version}")
 		(company "${project_creator}")
@@
 		(in_pos_files yes)
 		(dnp no)
-		(property "Reference" "X17"
+		(property "Reference" "X18"
 			(at 203.835 55.8801 0)
 			(show_name no)
@@
 			(project "BB3plus mainboard"
 				(path "/1df84e4f-233a-4f72-9418-c0020706bb76/9978f247-8f50-4e1a-a431-ff0e786a0608"
-					(reference "X17")
+					(reference "X18")
 					(unit 1)
 				)
@@
 		(in_pos_files yes)
 		(dnp no)
-		(property "Reference" "X16"
+		(property "Reference" "X17"
 			(at 125.095 34.925 0)
 			(show_name no)
@@
 			(project "BB3plus mainboard"
 				(path "/1df84e4f-233a-4f72-9418-c0020706bb76/9978f247-8f50-4e1a-a431-ff0e786a0608"
-					(reference "X16")
+					(reference "X17")
 					(unit 1)
 				)
@@
 		(in_pos_files yes)
 		(dnp no)
-		(property "Reference" "X18"
+		(property "Reference" "X19"
 			(at 269.875 55.88 0)
 			(show_name no)
@@
 			(project "BB3plus mainboard"
 				(path "/1df84e4f-233a-4f72-9418-c0020706bb76/9978f247-8f50-4e1a-a431-ff0e786a0608"
-					(reference "X18")
+					(reference "X19")
 					(unit 1)
 				)
@@
 		(dnp no)
 		(fields_autoplaced yes)
-		(property "Reference" "X15"
+		(property "Reference" "X16"
 			(at 120.65 158.7499 0)
 			(show_name no)
@@
 			(project "BB3plus mainboard"
 				(path "/1df84e4f-233a-4f72-9418-c0020706bb76/9978f247-8f50-4e1a-a431-ff0e786a0608"
-					(reference "X15")
+					(reference "X16")
 					(unit 1)
 				)

Commit message: #24
Parts:
- renumbered C128 to C126, C129 to C127, C130 to C128, C131 to C129, C132 to C130, C133 to C131, C134 to C132, C135 to C133, C136 to C134, C137 to C135, C138 to C136, D16 to D10, D15 to D9, IC24 to IC21, IC25 to IC22, IC26 to IC23, IC27 to IC24, JP20 to JP19, JP21 to JP20, R91 to R88, R92 to R89, R93 to R90, R94 to R91, R95 to R92

Commit message: USB CC wiring updated
Parts:
- IC22, IC24: LCSC (none) -> C38663
- renumbered R88 to R89, R89 to R90, R90 to R91, R91 to R92, R92 to R93
Changed lines of the file:
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@@
 	(title_block
 		(title "${project_name}")
-		(date "2026-10-12")
+		(date "2026-10-14")
 		(rev "${project_version}")
 		(company "${project_creator}")
@@
 		(in_pos_files yes)
 		(dnp no)
-		(property "Reference" "#GND045"
+		(property "Reference" "#GND046"
 			(at 261.62 91.44 0)
 			(hide yes)
@@
 			(project "BB3plus mainboard"
 				(path "/1df84e4f-233a-4f72-9418-c0020706bb76/9978f247-8f50-4e1a-a431-ff0e786a0608"
-					(reference "#GND045")
+					(reference "#GND046")
 					(unit 1)
 				)
@@
 		(in_pos_files yes)
 		(dnp no)
-		(property "Reference" "#GND042"
+		(property "Reference" "#GND043"
 			(at 182.88 91.44 0)
 			(hide yes)
@@
 			(project "BB3plus mainboard"
 				(path "/1df84e4f-233a-4f72-9418-c0020706bb76/9978f247-8f50-4e1a-a431-ff0e786a0608"
-					(reference "#GND042")
+					(reference "#GND043")
 					(unit 1)
 				)
@@
 		(in_pos_files yes)
 		(dnp no)
-		(property "Reference" "#GND037"
+		(property "Reference" "#GND038"
 			(at 63.5 93.98 0)
 			(hide yes)
@@
 			(project "BB3plus mainboard"
 				(path "/1df84e4f-233a-4f72-9418-c0020706bb76/9978f247-8f50-4e1a-a431-ff0e786a0608"
-					(reference "#GND037")
+					(reference "#GND038")
 					(unit 1)
 				)
@@
 		(in_pos_files yes)
 		(dnp no)
-		(property "Reference" "R91"
+		(property "Reference" "R92"
 			(at 142.24 100.33 90)
 			(show_name no)
@@
 			(project "BB3plus mainboard"
 				(path "/1df84e4f-233a-4f72-9418-c0020706bb76/9978f247-8f50-4e1a-a431-ff0e786a0608"
-					(reference "R91")
+					(reference "R92")
 					(unit 1)
 				)
@@
 		(in_pos_files yes)
 		(dnp no)
-		(property "Reference" "R88"
+		(property "Reference" "R89"
 			(at 75.565 175.26 90)
 			(show_name no)
@@
 			(project "BB3plus mainboard"
 				(path "/1df84e4f-233a-4f72-9418-c0020706bb76/9978f247-8f50-4e1a-a431-ff0e786a0608"
-					(reference "R88")
+					(reference "R89")
 					(unit 1)
 				)
@@
 		(in_pos_files yes)
 		(dnp no)
-		(property "Reference" "R92"
+		(property "Reference" "R93"
 			(at 199.39 133.985 0)
 			(show_name no)
@@
 			(project "BB3plus mainboard"
 				(path "/1df84e4f-233a-4f72-9418-c0020706bb76/9978f247-8f50-4e1a-a431-ff0e786a0608"
-					(reference "R92")
+					(reference "R93")
 					(unit 1)
 				)
@@
 		(in_pos_files yes)
 		(dnp no)
-		(property "Reference" "#GND043"
+		(property "Reference" "#GND044"
 			(at 195.58 91.44 0)
 			(hide yes)
@@
 			(project "BB3plus mainboard"
 				(path "/1df84e4f-233a-4f72-9418-c0020706bb76/9978f247-8f50-4e1a-a431-ff0e786a0608"
-					(reference "#GND043")
+					(reference "#GND044")
 					(unit 1)
 				)
@@
 		(in_pos_files yes)
 		(dnp no)
-		(property "Reference" "#GND040"
+		(property "Reference" "#GND041"
 			(at 114.3 91.44 0)
 			(hide yes)
@@
 			(project "BB3plus mainboard"
 				(path "/1df84e4f-233a-4f72-9418-c0020706bb76/9978f247-8f50-4e1a-a431-ff0e786a0608"
-					(reference "#GND040")
+					(reference "#GND041")
 					(unit 1)
 				)
@@
 		(in_pos_files yes)
 		(dnp no)
-		(property "Reference" "R90"
+		(property "Reference" "R91"
 			(at 132.08 100.33 90)
 			(show_name no)
@@
 			(project "BB3plus mainboard"
 				(path "/1df84e4f-233a-4f72-9418-c0020706bb76/9978f247-8f50-4e1a-a431-ff0e786a0608"
-					(reference "R90")
+					(reference "R91")
 					(unit 1)
 				)
@@
 		(in_pos_files yes)
 		(dnp no)
-		(property "Reference" "#GND039"
+		(property "Reference" "#GND040"
 			(at 104.14 99.06 0)
 			(hide yes)
@@
 			(project "BB3plus mainboard"
 				(path "/1df84e4f-233a-4f72-9418-c0020706bb76/9978f247-8f50-4e1a-a431-ff0e786a0608"
-					(reference "#GND039")
+					(reference "#GND040")
 					(unit 1)
 				)
@@
 			)
 		)
+		(property "LCSC" "C38663"
+			(at 256.54 111.76 0)
+			(hide yes)
+			(show_name no)
+			(do_not_autoplace no)
+			(effects
+				(font
+					(size 0.889 0.889)
+				)
+			)
+		)
 		(pin "3"
 		)
@@
 		(in_pos_files yes)
 		(dnp no)
-		(property "Reference" "#GND036"
+		(property "Reference" "#GND037"
 			(at 25.4 96.52 0)
 			(hide yes)
@@
 			(project "BB3plus mainboard"
 				(path "/1df84e4f-233a-4f72-9418-c0020706bb76/9978f247-8f50-4e1a-a431-ff0e786a0608"
-					(reference "#GND036")
+					(reference "#GND037")
 					(unit 1)
 				)
@@
 		(in_pos_files yes)
 		(dnp no)
-		(property "Reference" "R89"
+		(property "Reference" "R90"
 			(at 85.725 172.72 90)
 			(show_name no)
@@
 			(project "BB3plus mainboard"
 				(path "/1df84e4f-233a-4f72-9418-c0020706bb76/9978f247-8f50-4e1a-a431-ff0e786a0608"
-					(reference "R89")
+					(reference "R90")
 					(unit 1)
 				)
@@
 			)
 		)
+		(property "LCSC" "C38663"
+			(at 215.9 127 0)
+			(hide yes)
+			(show_name no)
+			(do_not_autoplace no)
+			(effects
+				(font
+					(size 0.889 0.889)
+				)
+			)
+		)
 		(pin "3"
 		)
@@
 		(in_pos_files yes)
 		(dnp no)
-		(property "Reference" "#GND044"
+		(property "Reference" "#GND045"
 			(at 248.92 91.44 0)
 			(hide yes)
@@
 			(project "BB3plus mainboard"
 				(path "/1df84e4f-233a-4f72-9418-c0020706bb76/9978f247-8f50-4e1a-a431-ff0e786a0608"
-					(reference "#GND044")
+					(reference "#GND045")
 					(unit 1)
 				)
@@
 		(in_pos_files yes)
 		(dnp no)
-		(property "Reference" "#GND041"
+		(property "Reference" "#GND042"
 			(at 147.32 104.14 0)
 			(hide yes)
@@
 			(project "BB3plus mainboard"
 				(path "/1df84e4f-233a-4f72-9418-c0020706bb76/9978f247-8f50-4e1a-a431-ff0e786a0608"
-					(reference "#GND041")
+					(reference "#GND042")
 					(unit 1)
 				)
@@
 		(in_pos_files yes)
 		(dnp no)
-		(property "Reference" "#GND038"
+		(property "Reference" "#GND039"
 			(at 78.74 111.76 0)
 			(hide yes)
@@
 			(project "BB3plus mainboard"
 				(path "/1df84e4f-233a-4f72-9418-c0020706bb76/9978f247-8f50-4e1a-a431-ff0e786a0608"
-					(reference "#GND038")
+					(reference "#GND039")
 					(unit 1)
 				)

Commit message: DVID_PWR_FAULT added
Parts:
- added R89: 10K, PCM_EEZ_passives:R_0603_1608Metric, symbol PCM_EEZ_passives:R-EU
- renumbered R89 to R90, R90 to R91, R91 to R92, R92 to R93, R93 to R94
Connections:
- net +3V3: now also R89.1
- net ~{DVID_PWR_FAULT}: now reaches IC21.5 (~{FLT})
- net ~{DVID_PWR_FAULT}: now also R89.2
- no-connect marks 2 -> 1
Other:
- moved on the sheet: C126, IC21
