File: KiCad/BB3plus mainboard/video_outputs.kicad_sch (KiCad schematic)
At the start: 35 parts, among them IC21 TPS22948DCKR, IC22 SN74LVC1G3157DCK, IC23 LMK1C1106APWR, IC24 SN74LVC1G3157DCK, X16 MGB0A1-1CDDB005H, X17 SS-53000-002, X18 505110-2291, X19 505110-2291, Y3 ECS-TXO-32CSMV-100-AN-TR

Commit message: DVID_PWR_ON added
Parts:
- added R89: 10K, PCM_EEZ_passives:R_0603_1608Metric, symbol PCM_EEZ_passives:R-EU
- renumbered R89 to R90, R90 to R91, R91 to R92, R92 to R93, R93 to R94, R94 to R95
Connections:
- net +3V3: now also R89.1
- net +5V: no longer IC21.3 (ON)
- new net DVID_PWR_ON: IC21.3 (ON), R89.2
Other:
- moved on the sheet: C126, R90

Commit message: Rear USB & Ethernet updated
Parts:
- X19: now not fitted; now left out of the parts list
Connections:
- net GBE_TXRX_A+: now also L15.6 (D2-_IC); no longer L15.1 (D1+_CONN)
- net GBE_TXRX_A-: now also L15.7 (D2+_IC); no longer L15.2 (D1-_CONN)
- net GBE_TXRX_B+: now also L15.9 (D1-_IC); no longer L15.4 (D2+_CONN)
- net GBE_TXRX_B-: now also L15.10 (D1+_IC); no longer L15.5 (D2-_CONN)
- net GBE_TXRX_C+: now also L16.6 (D2-_IC); no longer L16.1 (D1+_CONN)
- net GBE_TXRX_C-: now also L16.7 (D2+_IC); no longer L16.2 (D1-_CONN)
- net GBE_TXRX_D+: now also L16.9 (D1-_IC); no longer L16.4 (D2+_CONN)
- net GBE_TXRX_D-: now also L16.10 (D1+_IC); no longer L16.5 (D2-_CONN)
- net TRD1+: now also L15.5 (D2-_CONN); no longer L15.10 (D1+_IC)
- net TRD1-: now also L15.4 (D2+_CONN); no longer L15.9 (D1-_IC)
- net TRD2+: now also L15.2 (D1-_CONN); no longer L15.7 (D2+_IC)
- net TRD2-: now also L15.1 (D1+_CONN); no longer L15.6 (D2-_IC)
- net TRD3+: now also L16.5 (D2-_CONN); no longer L16.10 (D1+_IC)
- net TRD3-: now also L16.4 (D2+_CONN); no longer L16.9 (D1-_IC)
- net TRD4+: now also L16.2 (D1-_CONN); no longer L16.7 (D2+_IC)
- net TRD4-: now also L16.1 (D1+_CONN); no longer L16.6 (D2-_IC)
Other:
- moved on the sheet: C128, X16A

Commit message: #28
Parts:
- renumbered JP19 to JP18, JP20 to JP19
Changed lines of the file:
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@@
 	(title_block
 		(title "${project_name}")
-		(date "2026-10-18")
+		(date "2026-10-19")
 		(rev "${project_version}")
 		(company "${project_creator}")
@@
 		(in_pos_files yes)
 		(dnp no)
-		(property "Reference" "JP19"
+		(property "Reference" "JP18"
 			(at 195.58 113.03 0)
 			(show_name no)
@@
 			(project "BB3plus mainboard"
 				(path "/1df84e4f-233a-4f72-9418-c0020706bb76/9978f247-8f50-4e1a-a431-ff0e786a0608"
-					(reference "JP19")
+					(reference "JP18")
 					(unit 1)
 				)
@@
 		(dnp no)
 		(fields_autoplaced yes)
-		(property "Reference" "JP20"
+		(property "Reference" "JP19"
 			(at 232.41 88.8999 0)
 			(show_name no)
@@
 			(project "BB3plus mainboard"
 				(path "/1df84e4f-233a-4f72-9418-c0020706bb76/9978f247-8f50-4e1a-a431-ff0e786a0608"
-					(reference "JP20")
+					(reference "JP19")
 					(unit 1)
 				)

Commit message: #29
Parts:
- JP18: Label REFCLK #5 -> REFCLK #4
Connections:
- net DIB4_REFCLK: now also IC24.4 (COM); no longer IC23.14 (Y1)
- net DIB5_REFCLK: now also IC23.3 (Y0); no longer IC24.4 (COM)
- net at IC24.3 (NC): now also IC23.14 (Y1); no longer IC23.3 (Y0)
- net REFCLK #5 renamed REFCLK #4
Changed lines of the file:
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@@
 	(title_block
 		(title "${project_name}")
-		(date "2026-10-21")
+		(date "2026-10-22")
 		(rev "${project_version}")
 		(company "${project_creator}")
@@
 		)
 	)
+	(wire
+		(pts
+			(xy 259.08 134.62) (xy 261.62 134.62)
+		)
+		(stroke
+			(width 0)
+			(type default)
+		)
+	)
 	(polyline
 		(pts
@@
 	(wire
 		(pts
-			(xy 261.62 124.46) (xy 261.62 132.08)
+			(xy 261.62 124.46) (xy 261.62 134.62)
 		)
 		(stroke
@@
 	(wire
 		(pts
+			(xy 259.08 132.08) (xy 266.7 132.08)
+		)
+		(stroke
+			(width 0)
+			(type default)
+		)
+	)
+	(wire
+		(pts
 			(xy 68.58 177.8) (xy 45.72 177.8)
 		)
@@
 		)
 	)
-	(wire
-		(pts
-			(xy 259.08 134.62) (xy 266.7 134.62)
-		)
-		(stroke
-			(width 0)
-			(type default)
-		)
-	)
 	(polyline
 		(pts
@@
 		)
 	)
-	(wire
-		(pts
-			(xy 261.62 132.08) (xy 259.08 132.08)
-		)
-		(stroke
-			(width 0)
-			(type default)
-		)
-	)
 	(polyline
 		(pts
@@
 		)
 	)
-	(label "REFCLK #5"
+	(label "REFCLK #4"
 		(at 233.68 114.3 0)
 		(effects
@@
 		)
 	)
-	(global_label "DIB5_REFCLK"
+	(global_label "DIB4_REFCLK"
 		(shape bidirectional)
 		(at 269.24 106.68 0)
@@
 		)
 	)
+	(global_label "DIB5_REFCLK"
+		(shape output)
+		(at 266.7 132.08 0)
+		(fields_autoplaced yes)
+		(effects
+			(font
+				(size 0.889 0.889)
+			)
+			(justify left)
+		)
+		(property "Intersheetrefs" "${INTERSHEET_REFS}"
+			(at 277.0099 132.08 0)
+			(hide yes)
+			(show_name no)
+			(do_not_autoplace no)
+			(effects
+				(font
+					(size 1.27 1.27)
+				)
+				(justify left)
+			)
+		)
+	)
 	(global_label "DSI0_D0-"
 		(shape input)
@@
 		)
 	)
-	(global_label "DIB4_REFCLK"
-		(shape output)
-		(at 266.7 134.62 0)
-		(fields_autoplaced yes)
-		(effects
-			(font
-				(size 0.889 0.889)
-			)
-			(justify left)
-		)
-		(property "Intersheetrefs" "${INTERSHEET_REFS}"
-			(at 277.0099 134.62 0)
-			(hide yes)
-			(show_name no)
-			(do_not_autoplace no)
-			(effects
-				(font
-					(size 1.27 1.27)
-				)
-				(justify left)
-			)
-		)
-	)
 	(global_label "REAR_DVID_CEC"
 		(shape input)
@@
 			)
 		)
-		(property "Label" "REFCLK #5"
+		(property "Label" "REFCLK #4"
 			(at 195.58 116.84 0)
 			(show_name no)
