File: KiCad/BB3plus mainboard/digital_io_fan_encoder.kicad_sch (KiCad schematic)
At the start: 50 parts, among them IC10 EMC2301-1-ACZL-TR, IC11 ISO6763FDWR, IC12 BD00FC0W, IC13 THVD1420DR, IC14 TPD4E001DRLR, IC15 TPD4E001DRLR, SW2 PEC16-2215F-S0024, X12 22-27-2031, X13 TBP03R1-350-10BE

Commit message: #22
Parts:
- renumbered C64 to C63, C63 to C64
Other:
- moved on the sheet: C47, C49, C53, C55, C63, C65, C66, L6, R56, R57, R58, R59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

Commit message: TOUT connected
Parts:
- added JP20: (no value), PCM_EEZ_SMD:JP2 open (0603), symbol PCM_EEZ_unsorted:JP2 open
Connections:
- net RS485_TX_EN/DOUT2: now also JP20.2
- new net TOUT: JP20.1
Other:
- moved on the sheet: C48, C54, C58, C60, C61, C62, C64, IC11, IC13, IC14, IC15, L7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

Commit message: PE fault detection section updated
Parts:
- renumbered C47 to C48, C48 to C49, C49 to C50, C50 to C51, C51 to C52, C52 to C53, C53 to C54, C54 to C55, C55 to C56, C56 to C57, C57 to C58, C58 to C59, C59 to C60, C60 to C61, C61 to C62, C62 to C63, C63 to C64, C64 to C65, C65 to C66, C66 to C67, JP20 to JP11, R52 to R50, R53 to R51, R50 to R52, R51 to R53

Commit message: Various small changes
Parts:
- renumbered X12 to X13, X13 to X14
Changed lines of the file:
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@@
 	(title_block
 		(title "${project_name}")
-		(date "2026-10-09")
+		(date "2026-10-12")
 		(rev "${project_version}")
 		(company "${project_creator}")
@@
 	(wire
 		(pts
-			(xy 43.18 53.34) (xy 48.26 53.34)
+			(xy 30.48 53.34) (xy 48.26 53.34)
 		)
 		(stroke
@@
 	(wire
 		(pts
-			(xy 38.1 68.58) (xy 45.72 68.58)
+			(xy 30.48 68.58) (xy 45.72 68.58)
 		)
 		(stroke
@@
 	(global_label "RS485_RX{slash}DIN3"
 		(shape output)
-		(at 38.1 68.58 180)
+		(at 30.48 68.58 180)
 		(fields_autoplaced yes)
 		(effects
@@
 		)
 		(property "Intersheetrefs" "${INTERSHEET_REFS}"
-			(at 25.758 68.58 0)
+			(at 18.138 68.58 0)
 			(hide yes)
 			(show_name no)
@@
 	(global_label "RS485_TX{slash}DOUT3"
 		(shape input)
-		(at 43.18 53.34 180)
+		(at 30.48 53.34 180)
 		(fields_autoplaced yes)
 		(effects
@@
 		)
 		(property "Intersheetrefs" "${INTERSHEET_REFS}"
-			(at 29.8644 53.34 0)
+			(at 17.1644 53.34 0)
 			(hide yes)
 			(show_name no)
@@
 		(dnp no)
 		(fields_autoplaced yes)
-		(property "Reference" "X12"
+		(property "Reference" "X13"
 			(at 167.64 157.48 0)
 			(show_name no)
@@
 			(project "BB3plus mainboard"
 				(path "/1df84e4f-233a-4f72-9418-c0020706bb76/830c9101-e201-40d1-8c34-0dbed89b71c3"
-					(reference "X12")
+					(reference "X13")
 					(unit 1)
 				)
@@
 		(in_pos_files yes)
 		(dnp no)
-		(property "Reference" "X13"
+		(property "Reference" "X14"
 			(at 242.57 33.02 0)
 			(show_name no)
@@
 			(project "BB3plus mainboard"
 				(path "/1df84e4f-233a-4f72-9418-c0020706bb76/830c9101-e201-40d1-8c34-0dbed89b71c3"
-					(reference "X13")
+					(reference "X14")
 					(unit 1)
 				)

Commit message: #24
Parts:
- renumbered C48 to C46, C49 to C47, C50 to C48, C51 to C49, C52 to C50, C53 to C51, C54 to C52, C55 to C53, C56 to C54, C57 to C55, C58 to C56, C59 to C57, C60 to C58, C61 to C59, C62 to C60, C63 to C61, C64 to C62, C65 to C63, C66 to C64, C67 to C65, D13 to D7, IC13 to IC10, IC14 to IC11, IC15 to IC12, IC10 to IC7, IC11 to IC8, IC12 to IC9, JP11 to JP10, R46 to R43, R47 to R44, R48 to R45, R49 to R46, R50 to R47, R51 to R48, R52 to R49, R53 to R50, R54 to R51, R55 to R52, R56 to R53, R57 to R54, R58 to R55, R59 to R56
