File: KiCad/BB3plus mainboard/ac_dc_power.kicad_sch (KiCad schematic)
At the start: 99 parts, among them IC4 SN74HCS02PWR, IC5 TPS62933ODRLR, IC6 LM64460CPPQRYFRQ1, K1 AZ943-1CH-12DE, K2 AZ943-1CH-12DE, Q3 2N7002, Q4 2N7002, Q5 MMBT5401, Q6 DMP3013SFV-7, SW1 WBL2UOAGQR05CLR, X10 B3P-VH-FB-B, X11 B3P-VH-FB-B, X12 B3P-VH-FB-B, X5 571-0400, X6 GSP1.9101.1, X7 1-726388-2, X8 B3P-VH-FB-B, X9 22-23-2031

Commit message: Rear USB & Ethernet updated
Parts:
- renumbered TP8 to TP10, TP9 to TP11, TP10 to TP12, TP4 to TP6, TP5 to TP7, TP6 to TP8, TP7 to TP9
Changed lines of the file:
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@@
 		(in_bom no)
 		(on_board yes)
-		(in_pos_files yes)
+		(in_pos_files no)
 		(dnp no)
-		(property "Reference" "TP10"
+		(property "Reference" "TP12"
 			(at 259.08 140.335 90)
 			(show_name no)
@@
 			)
 		)
+		(property "DigiKey" ""
+			(at 259.08 142.24 0)
+			(hide yes)
+			(show_name no)
+			(do_not_autoplace no)
+			(effects
+				(font
+					(size 0.889 0.889)
+				)
+			)
+		)
+		(property "Mouser" ""
+			(at 259.08 142.24 0)
+			(hide yes)
+			(show_name no)
+			(do_not_autoplace no)
+			(effects
+				(font
+					(size 0.889 0.889)
+				)
+			)
+		)
+		(property "TME" ""
+			(at 259.08 142.24 0)
+			(hide yes)
+			(show_name no)
+			(do_not_autoplace no)
+			(effects
+				(font
+					(size 0.889 0.889)
+				)
+			)
+		)
+		(property "LCSC" ""
+			(at 259.08 142.24 0)
+			(hide yes)
+			(show_name no)
+			(do_not_autoplace no)
+			(effects
+				(font
+					(size 0.889 0.889)
+				)
+			)
+		)
 		(pin "1"
 		)
@@
 			(project "BB3plus mainboard"
 				(path "/1df84e4f-233a-4f72-9418-c0020706bb76/451f238c-56e9-49de-804a-2a19deb9fc4a"
-					(reference "TP10")
+					(reference "TP12")
 					(unit 1)
 				)
@@
 		(in_bom no)
 		(on_board yes)
-		(in_pos_files yes)
+		(in_pos_files no)
 		(dnp no)
-		(property "Reference" "TP9"
+		(property "Reference" "TP11"
 			(at 259.08 89.535 90)
 			(show_name no)
@@
 			)
 		)
+		(property "DigiKey" ""
+			(at 259.08 91.44 0)
+			(hide yes)
+			(show_name no)
+			(do_not_autoplace no)
+			(effects
+				(font
+					(size 0.889 0.889)
+				)
+			)
+		)
+		(property "Mouser" ""
+			(at 259.08 91.44 0)
+			(hide yes)
+			(show_name no)
+			(do_not_autoplace no)
+			(effects
+				(font
+					(size 0.889 0.889)
+				)
+			)
+		)
+		(property "TME" ""
+			(at 259.08 91.44 0)
+			(hide yes)
+			(show_name no)
+			(do_not_autoplace no)
+			(effects
+				(font
+					(size 0.889 0.889)
+				)
+			)
+		)
+		(property "LCSC" ""
+			(at 259.08 91.44 0)
+			(hide yes)
+			(show_name no)
+			(do_not_autoplace no)
+			(effects
+				(font
+					(size 0.889 0.889)
+				)
+			)
+		)
 		(pin "1"
 		)
@@
 			(project "BB3plus mainboard"
 				(path "/1df84e4f-233a-4f72-9418-c0020706bb76/451f238c-56e9-49de-804a-2a19deb9fc4a"
-					(reference "TP9")
+					(reference "TP11")
 					(unit 1)
 				)
@@
 		(in_bom no)
 		(on_board yes)
-		(in_pos_files yes)
+		(in_pos_files no)
 		(dnp no)
-		(property "Reference" "TP4"
+		(property "Reference" "TP6"
 			(at 93.345 86.995 0)
 			(show_name no)
@@
 			(project "BB3plus mainboard"
 				(path "/1df84e4f-233a-4f72-9418-c0020706bb76/451f238c-56e9-49de-804a-2a19deb9fc4a"
-					(reference "TP4")
+					(reference "TP6")
 					(unit 1)
 				)
@@
 		(in_pos_files yes)
 		(dnp no)
-		(property "Reference" "TP7"
+		(property "Reference" "TP9"
 			(at 104.14 70.485 90)
 			(show_name no)
@@
 			(project "BB3plus mainboard"
 				(path "/1df84e4f-233a-4f72-9418-c0020706bb76/451f238c-56e9-49de-804a-2a19deb9fc4a"
-					(reference "TP7")
+					(reference "TP9")
 					(unit 1)
 				)
@@
 		(in_bom no)
 		(on_board yes)
-		(in_pos_files yes)
+		(in_pos_files no)
 		(dnp no)
-		(property "Reference" "TP5"
+		(property "Reference" "TP7"
 			(at 93.345 89.535 0)
 			(show_name no)
@@
 			(project "BB3plus mainboard"
 				(path "/1df84e4f-233a-4f72-9418-c0020706bb76/451f238c-56e9-49de-804a-2a19deb9fc4a"
-					(reference "TP5")
+					(reference "TP7")
 					(unit 1)
 				)
@@
 		(in_bom no)
 		(on_board yes)
-		(in_pos_files yes)
+		(in_pos_files no)
 		(dnp no)
-		(property "Reference" "TP8"
+		(property "Reference" "TP10"
 			(at 149.225 169.545 90)
 			(show_name no)
@@
 			)
 		)
+		(property "DigiKey" ""
+			(at 147.32 172.72 0)
+			(hide yes)
+			(show_name no)
+			(do_not_autoplace no)
+			(effects
+				(font
+					(size 0.889 0.889)
+				)
+			)
+		)
+		(property "Mouser" ""
+			(at 147.32 172.72 0)
+			(hide yes)
+			(show_name no)
+			(do_not_autoplace no)
+			(effects
+				(font
+					(size 0.889 0.889)
+				)
+			)
+		)
+		(property "TME" ""
+			(at 147.32 172.72 0)
+			(hide yes)
+			(show_name no)
+			(do_not_autoplace no)
+			(effects
+				(font
+					(size 0.889 0.889)
+				)
+			)
+		)
+		(property "LCSC" ""
+			(at 147.32 172.72 0)
+			(hide yes)
+			(show_name no)
+			(do_not_autoplace no)
+			(effects
+				(font
+					(size 0.889 0.889)
+				)
+			)
+		)
 		(pin "1"
 		)
@@
 			(project "BB3plus mainboard"
 				(path "/1df84e4f-233a-4f72-9418-c0020706bb76/451f238c-56e9-49de-804a-2a19deb9fc4a"
-					(reference "TP8")
+					(reference "TP10")
 					(unit 1)
 				)
@@
 		(in_bom no)
 		(on_board yes)
-		(in_pos_files yes)
+		(in_pos_files no)
 		(dnp no)
-		(property "Reference" "TP6"
+		(property "Reference" "TP8"
 			(at 93.345 92.075 0)
 			(show_name no)
@@
 			(project "BB3plus mainboard"
 				(path "/1df84e4f-233a-4f72-9418-c0020706bb76/451f238c-56e9-49de-804a-2a19deb9fc4a"
-					(reference "TP6")
+					(reference "TP8")
 					(unit 1)
 				)

Commit message: SW1 footprint expanded
Parts:
- SW1: footprint PCM_EEZ_unsorted:WBL2UOAGQR05CLR -> PCM_EEZ_unsorted:WBL2UOAGQR05CLR_2
Changed lines of the file:
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@@
 	(title_block
 		(title "${project_name}")
-		(date "2026-10-15")
+		(date "2026-10-16")
 		(rev "${project_version}")
 		(company "${project_creator}")
@@
 			)
 		)
-		(property "Footprint" "PCM_EEZ_unsorted:WBL2UOAGQR05CLR"
-			(at 78.74 132.08 0)
+		(property "Footprint" "PCM_EEZ_unsorted:WBL2UOAGQR05CLR_2"
+			(at 78.74 137.16 0)
 			(hide yes)
 			(show_name no)
@@
 		)
 		(property "Description" "Illuminated push button switch"
-			(at 78.74 141.732 0)
+			(at 78.74 139.7 0)
 			(hide yes)
 			(show_name no)
@@
 			)
 		)
-		(property "Footprint" "PCM_EEZ_unsorted:WBL2UOAGQR05CLR"
-			(at 58.42 109.22 0)
+		(property "Footprint" "PCM_EEZ_unsorted:WBL2UOAGQR05CLR_2"
+			(at 63.5 109.22 0)
 			(hide yes)
 			(show_name no)
@@
 		)
 		(property "Description" "Illuminated push button switch"
-			(at 68.072 109.22 0)
+			(at 66.04 109.22 0)
 			(hide yes)
 			(show_name no)

Commit message: BOM updated
Parts:
- VAR1, VAR2, VAR3: value ERZE14A431 -> B72214S0271K101; DigiKey P16688-ND -> 495-76433-1-ND; LCSC C1527395 -> C7502584; Mouser 667-ERZ-E11A431 -> 871-B72214S271K101; TME V275LA20AP -> B72214S0271K101
Changed lines of the file:
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@@
 	(title_block
 		(title "${project_name}")
-		(date "2026-10-16")
+		(date "2026-10-18")
 		(rev "${project_version}")
 		(company "${project_creator}")
@@
 			)
 		)
-		(property "Value" "ERZE14A431"
+		(property "Value" "B72214S0271K101"
 			(at 86.36 36.195 90)
 			(show_name no)
@@
 			)
 		)
-		(property "DigiKey" "P16688-ND"
+		(property "DigiKey" "495-76433-1-ND"
 			(at 81.28 35.56 0)
 			(hide yes)
@@
 			)
 		)
-		(property "Mouser" "667-ERZ-E11A431"
+		(property "Mouser" "871-B72214S271K101"
 			(at 78.74 35.56 0)
 			(hide yes)
@@
 			)
 		)
-		(property "TME" "V275LA20AP"
+		(property "TME" "B72214S0271K101"
 			(at 76.2 35.56 0)
 			(hide yes)
@@
 			)
 		)
-		(property "LCSC" "C1527395"
+		(property "LCSC" "C7502584"
 			(at 88.9 35.56 90)
 			(hide yes)
@@
 			)
 		)
-		(property "Value" "ERZE14A431"
+		(property "Value" "B72214S0271K101"
 			(at 76.2 31.75 90)
 			(show_name no)
@@
 			)
 		)
-		(property "DigiKey" "P16688-ND"
+		(property "DigiKey" "495-76433-1-ND"
 			(at 81.28 30.48 0)
 			(hide yes)
@@
 			)
 		)
-		(property "Mouser" "667-ERZ-E11A431"
+		(property "Mouser" "871-B72214S271K101"
 			(at 83.82 30.48 0)
 			(hide yes)
@@
 			)
 		)
-		(property "TME" "V275LA20AP"
+		(property "TME" "B72214S0271K101"
 			(at 86.36 30.48 0)
 			(hide yes)
@@
 			)
 		)
-		(property "LCSC" "C1527395"
+		(property "LCSC" "C7502584"
 			(at 73.66 30.48 90)
 			(hide yes)
@@
 			)
 		)
-		(property "Value" "ERZE14A431"
+		(property "Value" "B72214S0271K101"
 			(at 76.2 45.085 90)
 			(show_name no)
@@
 			)
 		)
-		(property "DigiKey" "P16688-ND"
+		(property "DigiKey" "495-76433-1-ND"
 			(at 81.28 43.18 0)
 			(hide yes)
@@
 			)
 		)
-		(property "Mouser" "667-ERZ-E11A431"
+		(property "Mouser" "871-B72214S271K101"
 			(at 83.82 43.18 0)
 			(hide yes)
@@
 			)
 		)
-		(property "TME" "V275LA20AP"
+		(property "TME" "B72214S0271K101"
 			(at 86.36 43.18 0)
 			(hide yes)
@@
 			)
 		)
-		(property "LCSC" "C1527395"
+		(property "LCSC" "C7502584"
 			(at 73.66 43.18 90)
 			(hide yes)

Commit message: Wire harness added, BOM updated
Parts:
- X7: now not fitted; now left out of the parts list
Changed lines of the file:
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@@
 	(title_block
 		(title "${project_name}")
-		(date "2026-10-19")
+		(date "2026-10-21")
 		(rev "${project_version}")
 		(company "${project_creator}")
@@
 		(body_style 1)
 		(exclude_from_sim no)
-		(in_bom yes)
+		(in_bom no)
 		(on_board yes)
-		(in_pos_files yes)
-		(dnp no)
+		(in_pos_files no)
+		(dnp yes)
 		(property "Reference" "X7"
 			(at 29.845 36.195 0)

Commit message: #31
Changed lines of the file:
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@@
 		(exclude_from_sim no)
 		(at 215.265 24.765 0)
-		(size 60.325 16.51)
+		(size 60.325 18.415)
 		(margins 0.9525 0.9525 0.9525 0.9525)
 		(stroke
 			(width 0)
-			(type solid)
+			(type dot)
 			(color 132 0 132 1)
 		)

Commit message: PCB layout and BOM updated
Parts:
- R28, R29: footprint PCM_EEZ_passives:R_1210_3225Metric -> PCM_EEZ_passives:R_2010_5025Metric; TME CQ1210-100K-1% -> 201007J0104T4E
Changed lines of the file:
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@@
 			)
 		)
-		(property "Footprint" "PCM_EEZ_passives:R_1210_3225Metric"
+		(property "Footprint" "PCM_EEZ_passives:R_2010_5025Metric"
 			(at 91.44 180.34 0)
 			(hide yes)
@@
 			)
 		)
-		(property "TME" "CQ1210-100K-1%"
+		(property "TME" "201007J0104T4E"
 			(at 91.44 180.34 0)
 			(hide yes)
@@
 			)
 		)
-		(property "Footprint" "PCM_EEZ_passives:R_1210_3225Metric"
+		(property "Footprint" "PCM_EEZ_passives:R_2010_5025Metric"
 			(at 81.28 180.34 0)
 			(hide yes)
@@
 			)
 		)
-		(property "TME" "CQ1210-100K-1%"
+		(property "TME" "201007J0104T4E"
 			(at 81.28 180.34 0)
 			(hide yes)
